File: PCBs/left_board/left_board.kicad_sch (KiCad schematic)
At the start: 82 parts, among them J101 USB4510-03-1-A, J102 Conn_ARM_SWD_TagConnect_TC2030, J103 GSB12J21C1EU, J104 USB4510-03-1-A, SW101 SW_DIP_x01, SW102 SW_DIP_x01, SW103 SW_DIP_x01, SW104 SW_DIP_x01, SW105 SW_DIP_x01, SW106 SW_DIP_x01, SW107 SW_DIP_x01, SW108 SW_DIP_x01, SW109 SW_DIP_x01, SW110 SW_DIP_x01, SW111 SW_DIP_x01, SW112 SW_DIP_x01, SW113 SW_DIP_x01, SW114 SW_DIP_x01, SW115 SW_DIP_x01, SW116 SW_DIP_x01, SW117 SW_DIP_x01, SW118 SW_DIP_x01, SW119 SW_DIP_x01, SW120 SW_DIP_x01, SW121 SW_DIP_x01, SW122 SW_DIP_x01, SW123 SW_DIP_x01, SW124 SW_DIP_x01, SW125 SW_DIP_x01, SW126 SW_DIP_x01, SW127 SW_DIP_x01, SW128 RIC11-31S15.5D7-TH, U101 STM32G0C1CEUx, U102 USB2533-1080AEN, U103 M24256X-FCU6T_VF, U104 USBLC6-4SC6, U105 USBLC6-4SC6, U106 USBLC6-4SC6, Y101 CX2016SA24000D0HLLG3

Commit message: Left board routing half done
Connections:
- net +3V3 is gone; now on net +3.3V: R101.1, R102.1, U101.4 (VBAT), U101.6 (VDD), U102.10 (VDDA33_1), U102.15 (VDD33_1), U102.23 (VDD33_2), U102.26 (RESET_N), U102.29 (VDDA33_2), U102.36 (VDDA33_3), U103.A1 (VCC)
- net ENC_A: now also U101.43 (PB4)
- net ENC_B: now also U101.44 (PB5)
- net ENC_SW: now also U101.45 (PB6)
- net KEY_B3: no longer SW106.2
- net KEY_C3: no longer SW107.2
- net KEY_D1: now also U101.8 (PF0)
- net KEY_D3: now also U101.11 (PA0); no longer SW108.2
- net KEY_D4: now also SW126.2, U101.12 (PA1); no longer SW116.2
- net KEY_D5: now also SW127.2, U101.13 (PA2); no longer SW120.2
- net KEY_D6: now also SW120.2; no longer SW124.2
- net KEY_E1: now also U101.1 (PC13)
- net KEY_E2: now also SW116.2, U101.48 (PB9); no longer SW126.2
- net KEY_E3: now also SW124.2, U101.47 (PB8); no longer SW127.2
- net LED1: now also U101.46 (PB7)
- net SCL: now also U101.25 (PB13)
- net SDA: now also U101.26 (PB14)
- net KEY_D2: now reaches U101.9 (PF1)
- net KEY_D2: now also SW108.2
- new net KEY_B2: SW106.2
- new net KEY_C2: SW107.2
Other:
- moved on the sheet: SW116, SW120, SW124, SW126, SW127

Commit message: Left board done
Parts:
- added C105: 1u, Capacitor_SMD:C_0402_1005Metric, symbol Device:C_Small
- added C106: 100n, Capacitor_SMD:C_0402_1005Metric, symbol Device:C_Small
- added D128, D129: WHITE, LED_SMD:LED_0402_1005Metric, symbol Device:LED_Small
- added R106, R107: 3k3, Resistor_SMD:R_0402_1005Metric, symbol Device:R_Small
Connections:
- net +3.3V: now also C105.1, C106.1
- net GND: now also C105.2, C106.2, R106.2, R107.2
- net KEY_A1: now also U101.20 (PB1)
- net KEY_A2: now also U101.22 (PB10)
- net KEY_A3: now also U101.24 (PB12)
- net KEY_A4: now also U101.30 (PC6)
- net KEY_A5: now also U101.31 (PC7)
- net KEY_A6: now also U101.32 (PA10/UCPD1_DBCC2)
- net KEY_B1: now also U101.16 (PA5)
- net KEY_B2: now also U101.17 (PA6)
- net KEY_B3: now also U101.18 (PA7)
- net KEY_B4: now also U101.19 (PB0)
- net KEY_B5: now also U101.23 (PB11)
- net KEY_B6: now also U101.37 (PA15)
- net KEY_C1: now also U101.11 (PA0)
- net KEY_C2: now also U101.12 (PA1)
- net KEY_C3: now also U101.13 (PA2)
- net KEY_C4: now also U101.14 (PA3)
- net KEY_C5: now also U101.21 (PB2)
- net KEY_C6: now also U101.39 (PD1)
- net KEY_D1: now also U101.2 (PC14); no longer U101.8 (PF0)
- net KEY_D2: now also U101.3 (PC15); no longer U101.9 (PF1)
- net KEY_D3: now also U101.8 (PF0); no longer U101.11 (PA0)
- net KEY_D4: now also U101.9 (PF1); no longer U101.12 (PA1)
- net KEY_D5: now also U101.15 (PA4); no longer U101.13 (PA2)
- net KEY_D6: now also U101.29 (PA9/UCPD1_DBCC1)
- net STAT1: now reaches U101.41 (PD3)
- net STAT1: now also D128.2 (A)
- net STAT2: now reaches U101.42 (PB3)
- net STAT2: now also D129.2 (A)
- new net STAT1_K: D128.1 (K), R106.1
- new net STAT2_K: D129.1 (K), R107.1

Commit message: Right board done, all components ordered
Connections:
- net GND: now also D128.1 (K), D129.1 (K); no longer R106.2, R107.2
- net STAT1: now also R106.1; no longer D128.2 (A)
- net STAT1_K: now also D128.2 (A), R106.2; no longer D128.1 (K), R106.1
- net STAT2: now also R107.2; no longer D129.2 (A)
- net STAT2_K: now also D129.2 (A); no longer D129.1 (K)
Other:
- moved on the sheet: D128, D129, R106, R107
Changed lines of the file:
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@@
 	(symbol
 		(lib_id "Device:LED_Small")
-		(at 119.38 157.48 90)
+		(at 119.38 170.18 90)
 		(unit 1)
 		(exclude_from_sim no)
@@
 		(fields_autoplaced yes)
 		(property "Reference" "D128"
-			(at 121.92 156.1464 90)
+			(at 121.92 168.8464 90)
 			(effects
 				(font
@@
 		)
 		(property "Value" "WHITE"
-			(at 121.92 158.6864 90)
+			(at 121.92 171.3864 90)
 			(effects
 				(font
@@
 		)
 		(property "Footprint" "LED_SMD:LED_0402_1005Metric"
-			(at 119.38 157.48 90)
+			(at 119.38 170.18 90)
 			(effects
 				(font
@@
 		)
 		(property "Datasheet" "~"
-			(at 119.38 157.48 90)
+			(at 119.38 170.18 90)
 			(effects
 				(font
@@
 		)
 		(property "Description" "Light emitting diode, small symbol"
-			(at 119.38 157.48 0)
+			(at 119.38 170.18 0)
 			(effects
 				(font
@@
 	(symbol
 		(lib_id "Device:R_Small")
-		(at 119.38 170.18 0)
+		(at 119.38 157.48 0)
 		(unit 1)
 		(exclude_from_sim no)
@@
 		(fields_autoplaced yes)
 		(property "Reference" "R106"
-			(at 121.92 168.9099 0)
+			(at 121.92 156.2099 0)
 			(effects
 				(font
@@
 		)
 		(property "Value" "3k3"
-			(at 121.92 171.4499 0)
+			(at 121.92 158.7499 0)
 			(effects
 				(font
@@
 		)
 		(property "Footprint" "Resistor_SMD:R_0402_1005Metric"
-			(at 119.38 170.18 0)
+			(at 119.38 157.48 0)
 			(effects
 				(font
@@
 		)
 		(property "Datasheet" "~"
-			(at 119.38 170.18 0)
+			(at 119.38 157.48 0)
 			(effects
 				(font
@@
 		)
 		(property "Description" "Resistor, small symbol"
-			(at 119.38 170.18 0)
+			(at 119.38 157.48 0)
 			(effects
 				(font
@@
 	(symbol
 		(lib_id "Device:R_Small")
-		(at 132.08 170.18 0)
+		(at 132.08 157.48 180)
 		(unit 1)
 		(exclude_from_sim no)
@@
 		(fields_autoplaced yes)
 		(property "Reference" "R107"
-			(at 134.62 168.9099 0)
+			(at 134.62 156.2099 0)
 			(effects
 				(font
 					(size 1.27 1.27)
 				)
-				(justify left)
+				(justify right)
 			)
 		)
 		(property "Value" "3k3"
-			(at 134.62 171.4499 0)
+			(at 134.62 158.7499 0)
 			(effects
 				(font
 					(size 1.27 1.27)
 				)
-				(justify left)
+				(justify right)
 			)
 		)
 		(property "Footprint" "Resistor_SMD:R_0402_1005Metric"
-			(at 132.08 170.18 0)
+			(at 132.08 157.48 0)
 			(effects
 				(font
@@
 		)
 		(property "Datasheet" "~"
-			(at 132.08 170.18 0)
+			(at 132.08 157.48 0)
 			(effects
 				(font
@@
 		)
 		(property "Description" "Resistor, small symbol"
-			(at 132.08 170.18 0)
+			(at 132.08 157.48 0)
 			(effects
 				(font
@@
 	(symbol
 		(lib_id "Device:LED_Small")
-		(at 132.08 157.48 90)
+		(at 132.08 170.18 90)
 		(unit 1)
 		(exclude_from_sim no)
@@
 		(fields_autoplaced yes)
 		(property "Reference" "D129"
-			(at 134.62 156.1464 90)
+			(at 134.62 168.8464 90)
 			(effects
 				(font
@@
 		)
 		(property "Value" "WHITE"
-			(at 134.62 158.6864 90)
+			(at 134.62 171.3864 90)
 			(effects
 				(font
@@
 		)
 		(property "Footprint" "LED_SMD:LED_0402_1005Metric"
-			(at 132.08 157.48 90)
+			(at 132.08 170.18 90)
 			(effects
 				(font
@@
 		)
 		(property "Datasheet" "~"
-			(at 132.08 157.48 90)
+			(at 132.08 170.18 90)
 			(effects
 				(font
@@
 		)
 		(property "Description" "Light emitting diode, small symbol"
-			(at 132.08 157.48 0)
+			(at 132.08 170.18 0)
 			(effects
 				(font

Commit message: Knobs work properly
Parts:
- R104: value 47k -> 100k
- R105: value 100k -> 47k
Changed lines of the file:
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@@
 			)
 		)
-		(property "Value" "100k"
+		(property "Value" "47k"
 			(at 248.92 161.2899 0)
 			(effects
@@
 			)
 		)
-		(property "Value" "47k"
+		(property "Value" "100k"
 			(at 248.92 171.4499 0)
 			(effects
