File: PCBs/right_board/right_board.kicad_sch (KiCad schematic)
At the start: 82 parts, among them J101 USB4510-03-1-A, J102 Conn_ARM_SWD_TagConnect_TC2030, J103 GSB12J21C1EU, J104 USB4510-03-1-A, SW101 SW_DIP_x01, SW102 SW_DIP_x01, SW103 SW_DIP_x01, SW104 SW_DIP_x01, SW105 SW_DIP_x01, SW106 SW_DIP_x01, SW107 SW_DIP_x01, SW108 SW_DIP_x01, SW109 SW_DIP_x01, SW110 SW_DIP_x01, SW111 SW_DIP_x01, SW112 SW_DIP_x01, SW113 SW_DIP_x01, SW114 SW_DIP_x01, SW115 SW_DIP_x01, SW116 SW_DIP_x01, SW117 SW_DIP_x01, SW118 SW_DIP_x01, SW119 SW_DIP_x01, SW120 SW_DIP_x01, SW121 SW_DIP_x01, SW122 SW_DIP_x01, SW123 SW_DIP_x01, SW124 SW_DIP_x01, SW125 SW_DIP_x01, SW126 SW_DIP_x01, SW127 SW_DIP_x01, SW128 RIC11-31S15.5D7-TH, U101 STM32G0C1CEUx, U102 USB2533-1080AEN, U103 M24256X-FCU6T_VF, U104 USBLC6-4SC6, U105 USBLC6-4SC6, U106 USBLC6-4SC6, Y101 CX2016SA24000D0HLLG3

Commit message: Right board done, all components ordered
Parts:
- added C105: 1u, Capacitor_SMD:C_0402_1005Metric, symbol Device:C_Small
- added C106: 100n, Capacitor_SMD:C_0402_1005Metric, symbol Device:C_Small
- added D128, D129: WHITE, LED_SMD:LED_0402_1005Metric, symbol Device:LED_Small
- added R106, R107: 3k3, Resistor_SMD:R_0402_1005Metric, symbol Device:R_Small
Connections:
- net +3V3 is gone; now on net +3.3V: R101.1, R102.1, U101.4 (VBAT), U101.6 (VDD), U102.10 (VDDA33_1), U102.15 (VDD33_1), U102.23 (VDD33_2), U102.26 (RESET_N), U102.29 (VDDA33_2), U102.36 (VDDA33_3), U103.A1 (VCC)
- net +3.3V: now also C105.1, C106.1
- net ENC_A: now also U101.37 (PA15)
- net ENC_B: now also U101.42 (PB3)
- net ENC_SW: now also U101.39 (PD1)
- net GND: now also C105.2, C106.2, D128.1 (K), D129.1 (K)
- net KEY_A1: now also U101.45 (PB6)
- net KEY_A2: now also U101.46 (PB7)
- net KEY_A3: now also U101.3 (PC15)
- net KEY_A4: now also U101.8 (PF0)
- net KEY_A5: now also U101.9 (PF1)
- net KEY_A6: now also U101.11 (PA0)
- net KEY_B1: now also U101.44 (PB5)
- net KEY_B3: now also U101.12 (PA1); no longer SW106.2
- net KEY_B4: now also U101.15 (PA4)
- net KEY_B5: now also U101.16 (PA5)
- net KEY_B6: now also U101.17 (PA6)
- net KEY_C1: now also U101.1 (PC13)
- net KEY_C3: now also U101.18 (PA7); no longer SW107.2
- net KEY_C4: now also U101.19 (PB0)
- net KEY_C5: now also U101.20 (PB1)
- net KEY_C6: now also U101.21 (PB2)
- net KEY_D1: now also U101.14 (PA3)
- net KEY_D3: now also U101.23 (PB11); no longer SW108.2
- net KEY_D4: now also U101.24 (PB12)
- net KEY_D5: now also U101.26 (PB14)
- net KEY_D6: now also U101.25 (PB13)
- net KEY_E1: now also U101.29 (PA9/UCPD1_DBCC1)
- net KEY_E2: now also SW127.2, U101.30 (PC6); no longer SW126.2
- net KEY_E3: now also SW126.2, U101.31 (PC7); no longer SW127.2
- net LED1: now also U101.32 (PA10/UCPD1_DBCC2)
- net SCL: now also U101.47 (PB8)
- net SDA: now also U101.48 (PB9)
- net KEY_C2: now reaches U101.13 (PA2)
- net KEY_C2: now also SW107.2
- net KEY_B2: now reaches U101.2 (PC14)
- net KEY_B2: now also SW106.2
- net KEY_D2: now reaches U101.22 (PB10)
- net KEY_D2: now also SW108.2
- net STAT2: now reaches U101.41 (PD3)
- net STAT2: now also R107.2
- net STAT1: now reaches U101.43 (PB4)
- net STAT1: now also R106.2
- new net STAT1_K: D128.2 (A), R106.1
- new net STAT2_K: D129.2 (A), R107.1
Other:
- moved on the sheet: SW101, SW102, SW103, SW104, SW105, SW106, SW107, SW108, SW109, SW110, SW111, SW112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

Commit message: Pinout updates
Connections:
- net KEY_A1 renamed KEY_A7
- net KEY_A2 renamed KEY_A8
- net KEY_A3 renamed KEY_A9
- net KEY_A4 renamed KEY_A10
- net KEY_A5 renamed KEY_A11
- net KEY_A6 renamed KEY_A12
- net KEY_B1 renamed KEY_B7
- net KEY_B2 renamed KEY_B8
- net KEY_B3 renamed KEY_B9
- net KEY_B4 renamed KEY_B10
- net KEY_B5 renamed KEY_B11
- net KEY_B6 renamed KEY_B12
- net KEY_C1 renamed KEY_C7
- net KEY_C2 renamed KEY_C8
- net KEY_C3 renamed KEY_C9
- net KEY_C4 renamed KEY_C10
- net KEY_C5 renamed KEY_C11
- net KEY_C6 renamed KEY_C12
- net KEY_D1 renamed KEY_D7
- net KEY_D2 renamed KEY_D8
- net KEY_D3 renamed KEY_D9
- net KEY_D4 renamed KEY_D10
- net KEY_D5 renamed KEY_D11
- net KEY_D6 renamed KEY_D12
- net KEY_E1 renamed KEY_E6
- net KEY_E2 renamed KEY_E5
- net KEY_E3 renamed KEY_E4
Changed lines of the file:
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@@
 		)
 	)
-	(label "KEY_E2"
+	(label "KEY_E5"
 		(at 152.4 195.58 0)
 		(fields_autoplaced yes)
@@
 		)
 	)
-	(label "KEY_D1"
+	(label "KEY_D7"
 		(at 226.06 175.26 180)
 		(fields_autoplaced yes)
@@
 		)
 	)
-	(label "KEY_E1"
+	(label "KEY_E6"
 		(at 208.28 142.24 0)
 		(fields_autoplaced yes)
@@
 		)
 	)
-	(label "KEY_A5"
+	(label "KEY_A11"
 		(at 350.52 83.82 180)
 		(fields_autoplaced yes)
@@
 		)
 	)
-	(label "KEY_D3"
+	(label "KEY_D9"
 		(at 279.4 121.92 180)
 		(fields_autoplaced yes)
@@
 		)
 	)
-	(label "KEY_C4"
+	(label "KEY_C10"
 		(at 226.06 210.82 180)
 		(fields_autoplaced yes)
@@
 		)
 	)
-	(label "KEY_C2"
+	(label "KEY_C8"
 		(at 226.06 172.72 180)
 		(fields_autoplaced yes)
@@
 		)
 	)
-	(label "KEY_B4"
+	(label "KEY_B10"
 		(at 314.96 96.52 180)
 		(fields_autoplaced yes)
@@
 		)
 	)
-	(label "KEY_A6"
+	(label "KEY_A12"
 		(at 226.06 167.64 180)
 		(fields_autoplaced yes)
@@
 		)
 	)
-	(label "KEY_C6"
+	(label "KEY_C12"
 		(at 226.06 215.9 180)
 		(fields_autoplaced yes)
@@
 		)
 	)
-	(label "KEY_C3"
+	(label "KEY_C9"
 		(at 226.06 185.42 180)
 		(fields_autoplaced yes)
@@
 		)
 	)
-	(label "KEY_A2"
+	(label "KEY_A8"
 		(at 243.84 83.82 180)
 		(fields_autoplaced yes)
@@
 		)
 	)
-	(label "KEY_B3"
+	(label "KEY_B9"
 		(at 279.4 96.52 180)
 		(fields_autoplaced yes)
@@
 		)
 	)
-	(label "KEY_C2"
+	(label "KEY_C8"
 		(at 243.84 109.22 180)
 		(fields_autoplaced yes)
@@
 		)
 	)
-	(label "KEY_A4"
+	(label "KEY_A10"
 		(at 152.4 172.72 0)
 		(fields_autoplaced yes)
@@
 		)
 	)
-	(label "KEY_E3"
+	(label "KEY_E4"
 		(at 152.4 198.12 0)
 		(fields_autoplaced yes)
@@
 		)
 	)
-	(label "KEY_C6"
+	(label "KEY_C12"
 		(at 386.08 109.22 180)
 		(fields_autoplaced yes)
@@
 		)
 	)
-	(label "KEY_A3"
+	(label "KEY_A9"
 		(at 279.4 83.82 180)
 		(fields_autoplaced yes)
@@
 		)
 	)
-	(label "KEY_A1"
+	(label "KEY_A7"
 		(at 208.28 83.82 180)
 		(fields_autoplaced yes)
@@
 		)
 	)
-	(label "KEY_D3"
+	(label "KEY_D9"
 		(at 226.06 238.76 180)
 		(fields_autoplaced yes)
@@
 		)
 	)
-	(label "KEY_B6"
+	(label "KEY_B12"
 		(at 386.08 96.52 180)
 		(fields_autoplaced yes)
@@
 		)
 	)
-	(label "KEY_B5"
+	(label "KEY_B11"
 		(at 226.06 180.34 180)
 		(fields_autoplaced yes)
@@
 		)
 	)
-	(label "KEY_A4"
+	(label "KEY_A10"
 		(at 314.96 83.82 180)
 		(fields_autoplaced yes)
@@
 		)
 	)
-	(label "KEY_A6"
+	(label "KEY_A12"
 		(at 386.08 83.82 180)
 		(fields_autoplaced yes)
@@
 		)
 	)
-	(label "KEY_A1"
+	(label "KEY_A7"
 		(at 226.06 226.06 180)
 		(fields_autoplaced yes)
@@
 		)
 	)
-	(label "KEY_C5"
+	(label "KEY_C11"
 		(at 350.52 109.22 180)
 		(fields_autoplaced yes)
@@
 		)
 	)
-	(label "KEY_B1"
+	(label "KEY_B7"
 		(at 226.06 223.52 180)
 		(fields_autoplaced yes)
@@
 		)
 	)
-	(label "KEY_A2"
+	(label "KEY_A8"
 		(at 226.06 228.6 180)
 		(fields_autoplaced yes)
@@
 		)
 	)
-	(label "KEY_B3"
+	(label "KEY_B9"
 		(at 226.06 170.18 180)
 		(fields_autoplaced yes)
@@
 		)
 	)
-	(label "KEY_C1"
+	(label "KEY_C7"
 		(at 208.28 109.22 180)
 		(fields_autoplaced yes)
@@
 		)
 	)
-	(label "KEY_B5"
+	(label "KEY_B11"
 		(at 350.52 96.52 180)
 		(fields_autoplaced yes)
@@
 		)
 	)
-	(label "KEY_B2"
+	(label "KEY_B8"
 		(at 152.4 203.2 0)
 		(fields_autoplaced yes)
@@
 		)
 	)
-	(label "KEY_E1"
+	(label "KEY_E6"
 		(at 226.06 190.5 180)
 		(fields_autoplaced yes)
@@
 		)
 	)
-	(label "KEY_B6"
+	(label "KEY_B12"
 		(at 226.06 182.88 180)
 		(fields_autoplaced yes)
@@
 		)
 	)
-	(label "KEY_D1"
+	(label "KEY_D7"
 		(at 208.28 121.92 180)
 		(fields_autoplaced yes)
@@
 		)
 	)
-	(label "KEY_D4"
+	(label "KEY_D10"
 		(at 314.96 121.92 180)
 		(fields_autoplaced yes)
@@
 		)
 	)
-	(label "KEY_D5"
+	(label "KEY_D11"
 		(at 350.52 121.92 180)
 		(fields_autoplaced yes)
@@
 		)
 	)
-	(label "KEY_E2"
+	(label "KEY_E5"
 		(at 172.72 142.24 0)
 		(fields_autoplaced yes)
@@
 		)
 	)
-	(label "KEY_D4"
+	(label "KEY_D10"
 		(at 226.06 241.3 180)
 		(fields_autoplaced yes)
@@
 		)
 	)
-	(label "KEY_C1"
+	(label "KEY_C7"
 		(at 152.4 200.66 0)
 		(fields_autoplaced yes)
@@
 		)
 	)
-	(label "KEY_D6"
+	(label "KEY_D12"
 		(at 226.06 243.84 180)
 		(fields_autoplaced yes)
@@
 		)
 	)
-	(label "KEY_D2"
+	(label "KEY_D8"
 		(at 243.84 121.92 180)
 		(fields_autoplaced yes)
@@
 		)
 	)
-	(label "KEY_C5"
+	(label "KEY_C11"
 		(at 226.06 213.36 180)
 		(fields_autoplaced yes)
@@
 		)
 	)
-	(label "KEY_B2"
+	(label "KEY_B8"
 		(at 243.84 96.52 180)
 		(fields_autoplaced yes)
@@
 		)
 	)
-	(label "KEY_A5"
+	(label "KEY_A11"
 		(at 152.4 175.26 0)
 		(fields_autoplaced yes)
@@
 		)
 	)
-	(label "KEY_B4"
+	(label "KEY_B10"
 		(at 226.06 177.8 180)
 		(fields_autoplaced yes)
@@
 		)
 	)
-	(label "KEY_C3"
+	(label "KEY_C9"
 		(at 279.4 109.22 180)
 		(fields_autoplaced yes)
@@
 		)
 	)
-	(label "KEY_E3"
+	(label "KEY_E4"
 		(at 137.16 142.24 0)
 		(fields_autoplaced yes)
@@
 		)
 	)
-	(label "KEY_D5"
+	(label "KEY_D11"
 		(at 226.06 246.38 180)
 		(fields_autoplaced yes)
@@
 		)
 	)
-	(label "KEY_C4"
+	(label "KEY_C10"
 		(at 314.96 109.22 180)
 		(fields_autoplaced yes)
@@
 		)
 	)
-	(label "KEY_D2"
+	(label "KEY_D8"
 		(at 226.06 236.22 180)
 		(fields_autoplaced yes)
@@
 		)
 	)
-	(label "KEY_B1"
+	(label "KEY_B7"
 		(at 208.28 96.52 180)
 		(fields_autoplaced yes)
@@
 		)
 	)
-	(label "KEY_A3"
+	(label "KEY_A9"
 		(at 152.4 205.74 0)
 		(fields_autoplaced yes)
@@
 		)
 	)
-	(label "KEY_D6"
+	(label "KEY_D12"
 		(at 386.08 121.92 180)
 		(fields_autoplaced yes)

Commit message: Knobs work properly
Parts:
- R104: value 47k -> 100k
- R105: value 100k -> 47k
Changed lines of the file:
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@@
 			)
 		)
-		(property "Value" "100k"
+		(property "Value" "47k"
 			(at 248.92 161.2899 0)
 			(effects
@@
 			)
 		)
-		(property "Value" "47k"
+		(property "Value" "100k"
 			(at 248.92 171.4499 0)
 			(effects
