File: PCBs/keyboard_v2/usb.kicad_sch (KiCad schematic)
At the start: 20 parts, among them J601 USB4510-03-1-A, J602 USB4510-03-1-A, J603 GSB12J21C1EU, U601 USBLC6-4SC6, U602 USBLC6-4SC6, U603 USBLC6-4SC6, U604 STM32G0B1KBUx, U605 USB2533-1080AEN, Y601 CX2016SA24000D0HLLG3

Commit message: V2 progress
Parts:
- renumbered C601 to C1501, C604 to C1504, C605 to C1505, C606 to C1506, C607 to C1507, C608 to C1508, J601 to J1501, J602 to J1502, J603 to J1503, R603 to R1503, R604 to R1504, R605 to R1505, R606 to R1506, U601 to U1501, U602 to U1502, U603 to U1503, U604 to U1504, U605 to U1505, Y601 to Y1501
Connections:
- net +3.3V is gone; now on net +3V3: C1501.1, C602.1
- net +3V3: now also U1504.4 (VDD)
- net GND: now also U1504.33 (VSS), U1504.5 (VSS)
- net SWCLK: now also U1504.25 (PA14)
- net SWDIO: now also U1504.24 (PA13)
- net USB0_CC1: now also U1504.18 (PA8)
- net USB0_CC2: now also U1504.17 (PB2)
- net USB1_CC1: now also U1504.26 (PA15)
- net USB1_CC2: now also U1504.28 (PB4)
- net RST: now reaches U1504.6 (PF2)
- no-connect marks 20 -> 16
Other:
- moved on the sheet: C1501, J1502, J1503, U1501, U1502

Commit message: V2 Progress
Connections:
- net USB3_DN renamed USB_DN
- net USB3_DP renamed USB_DP
Changed lines of the file:
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@@
 	(wire
 		(pts
-			(xy 124.46 63.5) (xy 137.16 63.5)
+			(xy 121.92 63.5) (xy 137.16 63.5)
 		)
 		(stroke
@@
 	(wire
 		(pts
-			(xy 124.46 66.04) (xy 137.16 66.04)
+			(xy 121.92 66.04) (xy 137.16 66.04)
 		)
 		(stroke
@@
 		)
 	)
+	(hierarchical_label "USB_DN"
+		(shape bidirectional)
+		(at 121.92 66.04 180)
+		(fields_autoplaced yes)
+		(effects
+			(font
+				(size 1.27 1.27)
+			)
+			(justify right)
+		)
+	)
 	(hierarchical_label "SWDIO"
 		(shape bidirectional)
@@
 		(fields_autoplaced yes)
 		(effects
+			(font
+				(size 1.27 1.27)
+			)
+			(justify right)
+		)
+	)
+	(hierarchical_label "USB_DP"
+		(shape bidirectional)
+		(at 121.92 63.5 180)
+		(fields_autoplaced yes)
+		(effects

Commit message: Display schematic done
Changed lines of the file:
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@@
-		)
-	)
-	(hierarchical_label "SCL"
-		(shape bidirectional)
-		(at 43.18 101.6 180)
-		(fields_autoplaced yes)
-		(effects
-			(font
-				(size 1.27 1.27)
-			)
-			(justify right)
-		)
-	)
-	(hierarchical_label "SDA"
-		(shape input)
-		(at 43.18 104.14 180)
-		(fields_autoplaced yes)
-		(effects
-			(font
-				(size 1.27 1.27)
-			)
-			(justify right)
 		)
 	)

Commit message: V2 Schematic mostly done
Parts:
- renumbered C602 to C1502
Changed lines of the file:
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@@
 	(wire
 		(pts
+			(xy 33.02 104.14) (xy 45.72 104.14)
+		)
+		(stroke
+			(width 0)
+			(type default)
+		)
+	)
+	(wire
+		(pts
 			(xy 142.24 144.78) (xy 142.24 147.32)
 		)
@@
 	(wire
 		(pts
+			(xy 33.02 106.68) (xy 45.72 106.68)
+		)
+		(stroke
+			(width 0)
+			(type default)
+		)
+	)
+	(wire
+		(pts
 			(xy 50.8 160.02) (xy 63.5 160.02)
 		)
@@
 		)
 	)
+	(label "SDA"
+		(at 33.02 104.14 0)
+		(fields_autoplaced yes)
+		(effects
+			(font
+				(size 1.27 1.27)
+			)
+			(justify left bottom)
+		)
+	)
 	(label "VBUS_DET"
 		(at 124.46 33.02 0)
@@
 		)
 	)
+	(label "SCL"
+		(at 33.02 106.68 0)
+		(fields_autoplaced yes)
+		(effects
+			(font
+				(size 1.27 1.27)
+			)
+			(justify left bottom)
+		)
+	)
 	(label "USB0_CC1"
 		(at 63.5 152.4 180)
@@
 		(on_board yes)
 		(dnp no)
-		(property "Reference" "C602"
+		(property "Reference" "C1502"
 			(at 104.14 116.2113 0)
 			(effects
@@
 		(instances
 			(project "keyboard_v2"
-				(path "/e2360b7f-be71-48d9-b398-9f8cd45479d6/b599252a-0e44-4760-9c79-385d4380db60/2fa754a4-db8f-4839-bd38-632dd798fa1f"
-					(reference "C602")
-					(unit 1)
-				)
 				(path "/e2360b7f-be71-48d9-b398-9f8cd45479d6/8d5749a2-4d36-4f17-8c57-9c8b87d773d6/3f6891f6-a1b6-4bde-ae5f-d2abc12d04a0"
 					(reference "C1502")
 					(unit 1)
 				)
+				(path "/e2360b7f-be71-48d9-b398-9f8cd45479d6/b599252a-0e44-4760-9c79-385d4380db60/2fa754a4-db8f-4839-bd38-632dd798fa1f"
+					(reference "C602")
+					(unit 1)
+				)
 			)
 		)
@@
 		(dnp no)
 		(fields_autoplaced yes)
-		(property "Reference" "#PWR0613"
+		(property "Reference" "#PWR01513"
 			(at 91.44 113.03 0)
 			(effects
@@
 		(instances
 			(project "keyboard_v2"
-				(path "/e2360b7f-be71-48d9-b398-9f8cd45479d6/b599252a-0e44-4760-9c79-385d4380db60/2fa754a4-db8f-4839-bd38-632dd798fa1f"
-					(reference "#PWR0613")
-					(unit 1)
-				)
 				(path "/e2360b7f-be71-48d9-b398-9f8cd45479d6/8d5749a2-4d36-4f17-8c57-9c8b87d773d6/3f6891f6-a1b6-4bde-ae5f-d2abc12d04a0"
 					(reference "#PWR01513")
 					(unit 1)
 				)
+				(path "/e2360b7f-be71-48d9-b398-9f8cd45479d6/b599252a-0e44-4760-9c79-385d4380db60/2fa754a4-db8f-4839-bd38-632dd798fa1f"
+					(reference "#PWR0613")
+					(unit 1)
+				)
