File: PCBs/keyboard_v2/keyboard_v2.kicad_pcb (KiCad board)
At the start: 2 copper layers, 143.8 x 139.6 mm, 258 parts, among them J1501 USB4510-03-1-A, J1502 USB4510-03-1-A, J1503 GSB12J21C1EU, J601 USB4510-03-1-A, J602 USB4510-03-1-A, J603 GSB12J21C1EU, SW1201 SW_DIP_x01, SW1202 SW_DIP_x01, SW1203 SW_DIP_x01, SW1204 SW_DIP_x01, SW1205 SW_DIP_x01, SW1206 SW_DIP_x01, SW1207 SW_DIP_x01, SW1208 SW_DIP_x01, SW1209 SW_DIP_x01, SW1210 SW_DIP_x01, SW1211 SW_DIP_x01, SW1212 SW_DIP_x01, SW1213 SW_DIP_x01, SW1214 SW_DIP_x01, SW1215 SW_DIP_x01, SW1216 SW_DIP_x01, SW1217 SW_DIP_x01, SW1218 SW_DIP_x01, SW1219 SW_DIP_x01, SW1220 SW_DIP_x01, SW1221 SW_DIP_x01, SW1222 SW_DIP_x01, SW1223 SW_DIP_x01, SW1224 SW_DIP_x01, SW1225 SW_DIP_x01, SW1226 SW_DIP_x01, SW1227 RIC11-31S15.5D7-TH, SW1228 SW_DIP_x01, SW701 RIC11-31S15.5D7-TH, SW702 SW_DIP_x01, SW703 SW_DIP_x01, SW704 SW_DIP_x01, SW705 SW_DIP_x01, SW706 SW_DIP_x01, SW707 SW_DIP_x01, SW708 SW_DIP_x01, SW709 SW_DIP_x01, SW710 SW_DIP_x01, SW711 SW_DIP_x01, SW712 SW_DIP_x01, SW713 SW_DIP_x01, SW714 SW_DIP_x01, SW715 SW_DIP_x01, SW716 SW_DIP_x01, SW717 SW_DIP_x01, SW718 SW_DIP_x01, SW719 SW_DIP_x01, SW720 SW_DIP_x01, SW721 SW_DIP_x01, SW722 SW_DIP_x01, SW723 SW_DIP_x01, SW724 SW_DIP_x01, SW725 SW_DIP_x01, SW726 SW_DIP_x01, SW727 SW_DIP_x01, SW728 SW_DIP_x01, U1001 nRF52840-QFAA-F-R7, U1101 16B-WLCSP_2p34X2p43_RIT, U1301 STM32U5G9ZJJ6Q, U1501 USBLC6-4SC6, U1502 USBLC6-4SC6, U1503 USBLC6-4SC6, U1504 STM32G0B1KBUx, U1505 USB2533-1080AEN, U401 16B-WLCSP_2p34X2p43_RIT, U601 USBLC6-4SC6, U602 USBLC6-4SC6, U603 USBLC6-4SC6, U604 STM32G0B1KBUx, U605 USB2533-1080AEN, U801 STM32U5G9ZJJ6Q, U901 nRF52840-QFAA-F-R7, Y1301 16MHz, Y1501 CX2016SA24000D0HLLG3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

Commit message: V2 progress
Changed lines of the file:
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@@
 		(fp_arc
 			(start 48.00075 -53.5)
-			(mid 48.707889 -53.207124)
+			(mid 48.707854 -53.207118)
 			(end 49.00075 -52.5)
 			(stroke
@@
 		(fp_arc
 			(start 62.90075 -52.5)
-			(mid 63.193646 -53.207089)
+			(mid 63.19364 -53.207124)
 			(end 63.90075 -53.5)
 			(stroke
@@
 		(fp_arc
 			(start 65.450039 -53.499956)
-			(mid 66.157105 -53.207046)
+			(mid 66.15714 -53.207052)
 			(end 66.45 -52.499956)
 			(stroke
@@
 		(fp_arc
 			(start 66.45 52.499956)
-			(mid 66.157107 53.207048)
+			(mid 66.157101 53.207013)
 			(end 65.450039 53.499956)
 			(stroke
@@
 		(fp_arc
 			(start 63.90075 53.5)
-			(mid 63.19364 53.207095)
+			(mid 63.193676 53.207089)
 			(end 62.90075 52.5)
 			(stroke
@@
 		(fp_arc
 			(start 49.00075 52.5)
-			(mid 48.707883 53.207118)
+			(mid 48.707889 53.207154)
 			(end 48.00075 53.5)
 			(stroke

Commit message: V2 Progress
Parts:
- removed C1301, C1302, C801, C802: 6p, Capacitor_SMD:C_0402_1005Metric
- removed Y1301, Y801: 16MHz, Crystal:Crystal_SMD_2016-4Pin_2.0x1.6mm
- added C1003: 12p, Capacitor_SMD:C_0402_1005Metric, F.Cu at (-15.5, 62.0)
- added C1004: 12p, Capacitor_SMD:C_0402_1005Metric, F.Cu at (-15.5, 64.0)
- added C1005: 1p, Capacitor_SMD:C_0402_1005Metric, F.Cu at (-15.5, 65.9)
- added C1006: 1p2, Capacitor_SMD:C_0402_1005Metric, F.Cu at (-15.5, 67.9)
- added C1007: 100n, Capacitor_SMD:C_0402_1005Metric, F.Cu at (-15.5, 69.9)
- added C1008: 100n, Capacitor_SMD:C_0402_1005Metric, F.Cu at (-12.6, 62.0)
- added C1009: 100n, Capacitor_SMD:C_0402_1005Metric, F.Cu at (-12.6, 64.0)
- added C1010: 100n, Capacitor_SMD:C_0402_1005Metric, F.Cu at (-12.6, 65.9)
- added C1011: 100n, Capacitor_SMD:C_0402_1005Metric, F.Cu at (-12.6, 67.9)
- added C1012: 1u, Capacitor_SMD:C_0402_1005Metric, F.Cu at (-12.6, 69.9)
- added C1013: 100p, Capacitor_SMD:C_0402_1005Metric, F.Cu at (-9.75, 62.0)
- added C1014: 47n, Capacitor_SMD:C_0402_1005Metric, F.Cu at (-9.75, 64.0)
- added C1015: 1u, Capacitor_SMD:C_0402_1005Metric, F.Cu at (-9.75, 65.9)
- added C1323: 12p, Capacitor_SMD:C_0402_1005Metric, F.Cu at (-1.03, 75.6)
- added C1324: 12p, Capacitor_SMD:C_0402_1005Metric, F.Cu at (-1.03, 77.6)
- added C823: 12p, Capacitor_SMD:C_0402_1005Metric, F.Cu at (-15.5, 75.6)
- added C824: 12p, Capacitor_SMD:C_0402_1005Metric, F.Cu at (-15.5, 77.6)
- added C903: 12p, Capacitor_SMD:C_0402_1005Metric, F.Cu at (-1.03, 62.0)
- added C904: 12p, Capacitor_SMD:C_0402_1005Metric, F.Cu at (-1.03, 64.0)
- added C905: 1p, Capacitor_SMD:C_0402_1005Metric, F.Cu at (-1.03, 65.9)
- added C906: 1p2, Capacitor_SMD:C_0402_1005Metric, F.Cu at (-1.03, 67.9)
- added C907: 100n, Capacitor_SMD:C_0402_1005Metric, F.Cu at (-1.03, 69.9)
- added C908: 100n, Capacitor_SMD:C_0402_1005Metric, F.Cu at (1.84, 62.0)
- added C909: 100n, Capacitor_SMD:C_0402_1005Metric, F.Cu at (1.84, 64.0)
- added C910: 100n, Capacitor_SMD:C_0402_1005Metric, F.Cu at (1.84, 65.9)
- added C911: 100n, Capacitor_SMD:C_0402_1005Metric, F.Cu at (1.84, 67.9)
- added C912: 1u, Capacitor_SMD:C_0402_1005Metric, F.Cu at (1.84, 69.9)
- added C913: 100p, Capacitor_SMD:C_0402_1005Metric, F.Cu at (4.71, 62.0)
- added C914: 47n, Capacitor_SMD:C_0402_1005Metric, F.Cu at (4.71, 64.0)
- added C915: 1u, Capacitor_SMD:C_0402_1005Metric, F.Cu at (4.71, 65.9)
- added J1101: FH26W-27S-0.3SHW_60_, keyboard_footprints:FH26W27S03SHW60, F.Cu at (-10.6, 55.6)
- added J401: FH26W-27S-0.3SHW_60_, keyboard_footprints:FH26W27S03SHW60, F.Cu at (-11.9, 96.3)
- added L1001: 10u, Inductor_SMD:L_0402_1005Metric, F.Cu at (-6.86, 62.0)
- added L1002: 4n7, Inductor_SMD:L_0402_1005Metric, F.Cu at (-6.86, 64.0)
- added L1005: 2n2, Inductor_SMD:L_0402_1005Metric, F.Cu at (-6.86, 66.0)
- added L1006: 15n, Inductor_SMD:L_0402_1005Metric, F.Cu at (-6.86, 68.0)
- added L901: 10u, Inductor_SMD:L_0402_1005Metric, F.Cu at (7.60, 62.0)
- added L902: 4n7, Inductor_SMD:L_0402_1005Metric, F.Cu at (7.60, 64.0)
- added L905: 2n2, Inductor_SMD:L_0402_1005Metric, F.Cu at (7.60, 66.0)
- added L906: 15n, Inductor_SMD:L_0402_1005Metric, F.Cu at (7.60, 68.0)
- added Y1002: 32MHz, Crystal:Crystal_SMD_2016-4Pin_2.0x1.6mm, F.Cu at (-6.39, 70.8)
- added Y1302: 32MHz, Crystal:Crystal_SMD_2016-4Pin_2.0x1.6mm, F.Cu at (2.33, 76.4)
- added Y802: 32MHz, Crystal:Crystal_SMD_2016-4Pin_2.0x1.6mm, F.Cu at (-12.1, 76.4)
- added Y902: 32MHz, Crystal:Crystal_SMD_2016-4Pin_2.0x1.6mm, F.Cu at (8.07, 70.8)
- moved C1502 160.6 mm to (-6.77, 75.6)
- moved C602 143.6 mm to (7.69, 75.6)
Connections:
- AE1001 pad 1: unconnected-(AE1001-A-Pad1) -> /Left/Bluetooth/ANT
- AE901 pad 1: unconnected-(AE901-A-Pad1) -> /Right/Bluetooth/ANT
- C1501 pad 1: +3.3V -> +3V3
- C1502 pad 1: +3.3V -> +3V3
- C601 pad 1: +3.3V -> +3V3
- C602 pad 1: +3.3V -> +3V3
- SW702 pad 2: /Right/Keys Right/KEY_E4 -> /Right/Keys Right/KEY_E6
- SW712 pad 2: /Right/Keys Right/KEY_E6 -> /Right/Keys Right/KEY_E4
- U1001 pad 1: unconnected-(U1001-DEC1-Pad1) -> /Left/Bluetooth/DEC1
- U1001 pad 12: unconnected-(U1001-VDD_1-Pad12) -> Net-(U1001-VDD_1)
- U1001 pad 16: unconnected-(U1001-P0.18/NRESET-Pad16) -> /Left/Bluetooth/RST
- U1001 pad 17: unconnected-(U1001-VDD_2-Pad17) -> Net-(U1001-VDD_1)
- U1001 pad 25: unconnected-(U1001-VDD_3-Pad25) -> Net-(U1001-VDD_1)
- U1001 pad 26: unconnected-(U1001-SWDIO-Pad26) -> /Left/Bluetooth/SWDIO
- U1001 pad 27: unconnected-(U1001-SWDCLK-Pad27) -> /Left/Bluetooth/SWCLK
- U1001 pad 31: unconnected-(U1001-ANT-Pad31) -> /Left/Bluetooth/RF1
- U1001 pad 32: unconnected-(U1001-VSS_PA-Pad32) -> GND
- U1001 pad 33: unconnected-(U1001-DEC6-Pad33) -> /Left/Bluetooth/DEC4_6
- U1001 pad 34: unconnected-(U1001-DEC3-Pad34) -> /Left/Bluetooth/DEC3
- U1001 pad 35: unconnected-(U1001-XC1-Pad35) -> /Left/Bluetooth/XC1
- U1001 pad 36: unconnected-(U1001-XC2-Pad36) -> /Left/Bluetooth/XC2
- U1001 pad 37: unconnected-(U1001-VDD_4-Pad37) -> Net-(U1001-VDD_1)
- U1001 pad 45: unconnected-(U1001-VSS_1-Pad45) -> GND
- U1001 pad 46: unconnected-(U1001-DEC4-Pad46) -> /Left/Bluetooth/DEC4_6
- U1001 pad 47: unconnected-(U1001-DCC-Pad47) -> /Left/Bluetooth/DCC1
- U1001 pad 48: unconnected-(U1001-VDD_5-Pad48) -> Net-(U1001-VDD_1)
- U1001 pad 49: unconnected-(U1001-VSS_2-Pad49) -> GND
- U1504 pad 17: unconnected-(U1504-PB2-Pad17) -> /Left/USB/USB0_CC2
- U1504 pad 18: unconnected-(U1504-PA8-Pad18) -> /Left/USB/USB0_CC1
- U1504 pad 24: unconnected-(U1504-PA13-Pad24) -> /Left/USB/SWDIO
- U1504 pad 25: unconnected-(U1504-PA14-Pad25) -> /Left/USB/SWCLK
- U1504 pad 26: unconnected-(U1504-PA15-Pad26) -> /Left/USB/USB1_CC1
- U1504 pad 28: unconnected-(U1504-PB4-Pad28) -> /Left/USB/USB1_CC2
- U1504 pad 33: Net-(U1504-VSS-Pad33) -> GND
- U1504 pad 4: unconnected-(U1504-VDD-Pad4) -> +3V3
- U1504 pad 5: Net-(U1504-VSS-Pad33) -> GND
- U1504 pad 6: unconnected-(U1504-PF2-Pad6) -> /Left/USB/RST
- U604 pad 17: unconnected-(U604-PB2-Pad17) -> /Right/USB/USB0_CC2
- U604 pad 18: unconnected-(U604-PA8-Pad18) -> /Right/USB/USB0_CC1
- U604 pad 24: unconnected-(U604-PA13-Pad24) -> /Right/USB/SWDIO
- U604 pad 25: unconnected-(U604-PA14-Pad25) -> /Right/USB/SWCLK
- U604 pad 26: unconnected-(U604-PA15-Pad26) -> /Right/USB/USB1_CC1
- U604 pad 28: unconnected-(U604-PB4-Pad28) -> /Right/USB/USB1_CC2
- U604 pad 33: Net-(U604-VSS-Pad33) -> GND
- U604 pad 4: unconnected-(U604-VDD-Pad4) -> +3V3
- U604 pad 5: Net-(U604-VSS-Pad33) -> GND
- U604 pad 6: unconnected-(U604-PF2-Pad6) -> /Right/USB/RST
- U901 pad 1: unconnected-(U901-DEC1-Pad1) -> /Right/Bluetooth/DEC1
- U901 pad 12: unconnected-(U901-VDD_1-Pad12) -> Net-(U901-VDD_1)
- U901 pad 16: unconnected-(U901-P0.18/NRESET-Pad16) -> /Right/Bluetooth/RST
- U901 pad 17: unconnected-(U901-VDD_2-Pad17) -> Net-(U901-VDD_1)
- U901 pad 25: unconnected-(U901-VDD_3-Pad25) -> Net-(U901-VDD_1)
- U901 pad 26: unconnected-(U901-SWDIO-Pad26) -> /Right/Bluetooth/SWDIO
- U901 pad 27: unconnected-(U901-SWDCLK-Pad27) -> /Right/Bluetooth/SWCLK
- U901 pad 31: unconnected-(U901-ANT-Pad31) -> /Right/Bluetooth/RF1
- U901 pad 32: unconnected-(U901-VSS_PA-Pad32) -> GND
- U901 pad 33: unconnected-(U901-DEC6-Pad33) -> /Right/Bluetooth/DEC4_6
- U901 pad 34: unconnected-(U901-DEC3-Pad34) -> /Right/Bluetooth/DEC3
- U901 pad 35: unconnected-(U901-XC1-Pad35) -> /Right/Bluetooth/XC1
- U901 pad 36: unconnected-(U901-XC2-Pad36) -> /Right/Bluetooth/XC2
- U901 pad 37: unconnected-(U901-VDD_4-Pad37) -> Net-(U901-VDD_1)
- U901 pad 45: unconnected-(U901-VSS_1-Pad45) -> GND
- U901 pad 46: unconnected-(U901-DEC4-Pad46) -> /Right/Bluetooth/DEC4_6
- U901 pad 47: unconnected-(U901-DCC-Pad47) -> /Right/Bluetooth/DCC1
- U901 pad 48: unconnected-(U901-VDD_5-Pad48) -> Net-(U901-VDD_1)
- U901 pad 49: unconnected-(U901-VSS_2-Pad49) -> GND

Commit message: V2 Schematic mostly done
Parts:
- removed AE1001, AE901: Antenna, RF_Antenna:Texas_SWRA117D_2.4GHz_Left
- added AE202: Antenna_Shield, RF_Antenna:Texas_SWRA117D_2.4GHz_Left, F.Cu at (-11.8, 192.9)
- added AE302: Antenna_Shield, RF_Antenna:Texas_SWRA117D_2.4GHz_Right, F.Cu at (-20.9, 202.0)
- added IC1401: ADP5360ACBZ-2-R7, keyboard_footprints:ADP5360ACBZ1R7, F.Cu at (-27.0, 137.2)
- added IC501: ADP5360ACBZ-2-R7, keyboard_footprints:ADP5360ACBZ1R7, F.Cu at (-15.3, 137.2)
- added J201: TMS-115-01-G-S, keyboard_parts:debug_header, B.Cu at (191.4, 120.2)
- added J301: TMS-115-01-G-S, keyboard_parts:debug_header, F.Cu at (-24.3, 130.8)
- added Q1201: DMN21D2UFB-7B, keyboard_footprints:DMN21D2UFB7B, F.Cu at (-8.07, 126.2)
- added Q1401: DMP2104LP-7, keyboard_footprints:DMP2104LP7, F.Cu at (-27.8, 140.8)
- added Q501: DMP2104LP-7, keyboard_footprints:DMP2104LP7, F.Cu at (-16.1, 140.8)
- added Q701: DMN21D2UFB-7B, keyboard_footprints:DMN21D2UFB7B, F.Cu at (-8.07, 116.6)
- added R1201: 4k7, Resistor_SMD:R_0402_1005Metric, F.Cu at (-10.8, 126.2)
- added R1204: 100k, Resistor_SMD:R_0402_1005Metric, F.Cu at (-10.8, 128.2)
- added R1208: 100k, Resistor_SMD:R_0402_1005Metric, F.Cu at (-10.8, 130.2)
- added R701: 4k7, Resistor_SMD:R_0402_1005Metric, F.Cu at (-10.8, 116.6)
- added R708: 100k, Resistor_SMD:R_0402_1005Metric, F.Cu at (-10.8, 118.6)
- added R709: 100k, Resistor_SMD:R_0402_1005Metric, F.Cu at (-10.8, 120.5)
- added SW1402: PCM12SMTBR, keyboard_footprints:PCM12SMTBR, F.Cu at (-8.65, 155.1)
- added SW502: PCM12SMTBR, keyboard_footprints:PCM12SMTBR, F.Cu at (-8.65, 165.5)
- added TP1401: 3mm, TestPoint:TestPoint_Pad_D3.0mm, F.Cu at (-31.9, 137.4)
- added TP1402: 3mm, TestPoint:TestPoint_Pad_D3.0mm, F.Cu at (-31.9, 142.4)
- added TP501: 3mm, TestPoint:TestPoint_Pad_D3.0mm, F.Cu at (-20.2, 137.4)
- added TP502: 3mm, TestPoint:TestPoint_Pad_D3.0mm, F.Cu at (-20.2, 142.4)
- added U1302: M24256X-FCU6T_VF, keyboard_footprints:BGA4C50P2X2_70X98X33, F.Cu at (-41.5, 192.2)
- added U1401: MAX9938TEBS+TG45, keyboard_footprints:BGA4C50P2X2_100X100X67, F.Cu at (-28.0, 143.7)
- added U501: MAX9938TEBS+TG45, keyboard_footprints:BGA4C50P2X2_100X100X67, F.Cu at (-16.3, 143.7)
- added U802: M24256X-FCU6T_VF, keyboard_footprints:BGA4C50P2X2_70X98X33, F.Cu at (-36.7, 192.2)
Connections:
- C1007 pad 1: Net-(U1001-VDD_1) -> +1V8
- C1008 pad 1: Net-(U1001-VDD_1) -> +1V8
- C1009 pad 1: Net-(U1001-VDD_1) -> +1V8
- C1010 pad 1: Net-(U1001-VDD_1) -> +1V8
- C1012 pad 1: Net-(U1001-VDD_1) -> +1V8
- C1313 pad 1: +1V8 -> +3V3
- C1315 pad 1: +1V8 -> +3V3
- C813 pad 1: +1V8 -> +3V3
- C815 pad 1: +1V8 -> +3V3
- C907 pad 1: Net-(U901-VDD_1) -> +1V8
- C908 pad 1: Net-(U901-VDD_1) -> +1V8
- C909 pad 1: Net-(U901-VDD_1) -> +1V8
- C910 pad 1: Net-(U901-VDD_1) -> +1V8
- C912 pad 1: Net-(U901-VDD_1) -> +1V8
- J1101 pad 1: unconnected-(J1101-Pad1) -> /Left/Display/ELVSS
- J1101 pad 10: unconnected-(J1101-Pad10) -> /Left/Display/DSI_CKP
- J1101 pad 11: unconnected-(J1101-Pad11) -> /Left/Display/DSI_CKN
- J1101 pad 12: unconnected-(J1101-Pad12) -> GND
- J1101 pad 14: unconnected-(J1101-Pad14) -> GND
- J1101 pad 15: unconnected-(J1101-Pad15) -> GND
- J1101 pad 16: unconnected-(J1101-Pad16) -> /Left/Display/IM0
- J1101 pad 17: unconnected-(J1101-Pad17) -> +1V8
- J1101 pad 18: unconnected-(J1101-Pad18) -> GND
- J1101 pad 19: unconnected-(J1101-Pad19) -> /Left/Display/RST_DISP
- J1101 pad 2: unconnected-(J1101-Pad2) -> /Left/Display/ELVDD
- J1101 pad 20: unconnected-(J1101-Pad20) -> /Left/Display/DSI_TE
- J1101 pad 21: unconnected-(J1101-Pad21) -> /Left/Display/SWIRE
- J1101 pad 22: unconnected-(J1101-Pad22) -> GND
- J1101 pad 23: unconnected-(J1101-Pad23) -> +3V3
- J1101 pad 24: unconnected-(J1101-Pad24) -> /Left/Display/RST_TP
- J1101 pad 25: unconnected-(J1101-Pad25) -> /Left/Display/INT_TP
- J1101 pad 26: unconnected-(J1101-Pad26) -> /Left/Display/SCL_TP
- J1101 pad 27: unconnected-(J1101-Pad27) -> /Left/Display/SDA_TP
- J1101 pad 4: unconnected-(J1101-Pad4) -> /Left/Display/AVDD
- J1101 pad 5: unconnected-(J1101-Pad5) -> +1V8
- J1101 pad 6: unconnected-(J1101-Pad6) -> GND
- J1101 pad 7: unconnected-(J1101-Pad7) -> /Left/Display/DSI_D0P
- J1101 pad 8: unconnected-(J1101-Pad8) -> /Left/Display/DSI_D0N
- J1101 pad 9: unconnected-(J1101-Pad9) -> GND
- J1101 pad MP1: unconnected-(J1101-PadMP1) -> GND
- J1101 pad MP2: unconnected-(J1101-PadMP2) -> GND
- J401 pad 1: unconnected-(J401-Pad1) -> /Right/Display/ELVSS
- J401 pad 10: unconnected-(J401-Pad10) -> /Right/Display/DSI_CKP
- J401 pad 11: unconnected-(J401-Pad11) -> /Right/Display/DSI_CKN
- J401 pad 12: unconnected-(J401-Pad12) -> GND
- J401 pad 14: unconnected-(J401-Pad14) -> GND
- J401 pad 15: unconnected-(J401-Pad15) -> GND
- J401 pad 16: unconnected-(J401-Pad16) -> /Right/Display/IM0
- J401 pad 17: unconnected-(J401-Pad17) -> +1V8
- J401 pad 18: unconnected-(J401-Pad18) -> GND
- J401 pad 19: unconnected-(J401-Pad19) -> /Right/Display/RST_DISP
- J401 pad 2: unconnected-(J401-Pad2) -> /Right/Display/ELVDD
- J401 pad 20: unconnected-(J401-Pad20) -> /Right/Display/DSI_TE
- J401 pad 21: unconnected-(J401-Pad21) -> /Right/Display/SWIRE
- J401 pad 22: unconnected-(J401-Pad22) -> GND
- J401 pad 23: unconnected-(J401-Pad23) -> +3V3
- J401 pad 24: unconnected-(J401-Pad24) -> /Right/Display/RST_TP
- J401 pad 25: unconnected-(J401-Pad25) -> /Right/Display/INT_TP
- J401 pad 26: unconnected-(J401-Pad26) -> /Right/Display/SCL_TP
- J401 pad 27: unconnected-(J401-Pad27) -> /Right/Display/SDA_TP
- J401 pad 4: unconnected-(J401-Pad4) -> /Right/Display/AVDD
- J401 pad 5: unconnected-(J401-Pad5) -> +1V8
- J401 pad 6: unconnected-(J401-Pad6) -> GND
- J401 pad 7: unconnected-(J401-Pad7) -> /Right/Display/DSI_D0P
- J401 pad 8: unconnected-(J401-Pad8) -> /Right/Display/DSI_D0N
- J401 pad 9: unconnected-(J401-Pad9) -> GND
- J401 pad MP1: unconnected-(J401-PadMP1) -> GND
- J401 pad MP2: unconnected-(J401-PadMP2) -> GND
- R1301 pad 1: +3V3 -> +1V8
- R1302 pad 1: +3V3 -> +1V8
- R1401 pad 2: /Left/Power/BTN -> /Left/Main MCU Left/PWR_MR
- R501 pad 2: /Right/Power/BTN -> /Right/Main MCU Right/PWR_MR
- R801 pad 1: +3V3 -> +1V8
- R802 pad 1: +3V3 -> +1V8
- SW701 pad A: /Right/Keys Right/ENC_A -> /Right/Keys Right/ENC_B
- U1001 pad 12: Net-(U1001-VDD_1) -> +1V8
- U1001 pad 17: Net-(U1001-VDD_1) -> +1V8
- U1001 pad 25: Net-(U1001-VDD_1) -> +1V8
- U1001 pad 37: Net-(U1001-VDD_1) -> +1V8
- U1001 pad 48: Net-(U1001-VDD_1) -> +1V8
- U1301 pad E1: unconnected-(U1301B-DSI_D0N-PadE1) -> /Left/Display/DSI_D0N
- U1301 pad E2: unconnected-(U1301B-DSI_D0P-PadE2) -> /Left/Display/DSI_D0P
- U1301 pad E6: +1V8 -> +3V3
- U1301 pad F1: unconnected-(U1301B-DSI_CKN-PadF1) -> /Left/Display/DSI_CKN
- U1301 pad F2: unconnected-(U1301B-DSI_CKP-PadF2) -> /Left/Display/DSI_CKP
- U1301 pad H2: unconnected-(U1301B-PH0-OSC_IN-PadH2) -> /Left/Main MCU Left/OSC_IN
- U1301 pad J1: unconnected-(U1301B-PH1-OSC_OUT-PadJ1) -> /Left/Main MCU Left/OSC_OUT
- U1301 pad J2: unconnected-(U1301B-NRST-PadJ2) -> /Left/Main MCU Left/RST
- U1504 pad 6: /Left/USB/RST -> /Left/Main MCU Left/USB_RST
- U604 pad 6: /Right/USB/RST -> /Right/Main MCU Right/USB_RST
- U801 pad E1: unconnected-(U801B-DSI_D0N-PadE1) -> /Right/Display/DSI_D0N
- U801 pad E2: unconnected-(U801B-DSI_D0P-PadE2) -> /Right/Display/DSI_D0P
- U801 pad E6: +1V8 -> +3V3
- U801 pad F1: unconnected-(U801B-DSI_CKN-PadF1) -> /Right/Display/DSI_CKN
- U801 pad F2: unconnected-(U801B-DSI_CKP-PadF2) -> /Right/Display/DSI_CKP
- U801 pad H2: unconnected-(U801B-PH0-OSC_IN-PadH2) -> /Right/Main MCU Right/OSC_IN
- U801 pad J1: unconnected-(U801B-PH1-OSC_OUT-PadJ1) -> /Right/Main MCU Right/OSC_OUT
- U801 pad J2: unconnected-(U801B-NRST-PadJ2) -> /Right/Main MCU Right/RST
- U901 pad 12: Net-(U901-VDD_1) -> +1V8
- U901 pad 17: Net-(U901-VDD_1) -> +1V8
- U901 pad 25: Net-(U901-VDD_1) -> +1V8
- U901 pad 37: Net-(U901-VDD_1) -> +1V8
- U901 pad 48: Net-(U901-VDD_1) -> +1V8

Commit message: Schematic mostly done, moving onto PCB
Parts:
- removed C1318, C1320, C818, C820: 100n, Capacitor_SMD:C_0201_0603Metric
- removed the REF** at (295.0, 140.0)
- removed the REF** at (135.0, 140.0)
- added C1201: 100n, Capacitor_SMD:C_0402_1005Metric, F.Cu at (-73.8, 114.9)
- added C1202: 100n, Capacitor_SMD:C_0402_1005Metric, F.Cu at (-73.8, 116.9)
- added C1203: 100n, Capacitor_SMD:C_0402_1005Metric, F.Cu at (-73.8, 118.8)
- added C1204: 100n, Capacitor_SMD:C_0402_1005Metric, F.Cu at (-70.9, 114.9)
- added C1205: 100n, Capacitor_SMD:C_0402_1005Metric, F.Cu at (-70.9, 116.9)
- added C1206: 100n, Capacitor_SMD:C_0402_1005Metric, F.Cu at (-70.9, 118.8)
- added C1207: 100n, Capacitor_SMD:C_0402_1005Metric, F.Cu at (-68.1, 114.9)
- added C1208: 100n, Capacitor_SMD:C_0402_1005Metric, F.Cu at (-68.1, 116.9)
- added C1209: 100n, Capacitor_SMD:C_0402_1005Metric, F.Cu at (-68.1, 118.8)
- added C1301: 100n, Capacitor_SMD:C_0402_1005Metric, F.Cu at (17.9, 188.7)
- added C1302: 100n, Capacitor_SMD:C_0402_1005Metric, F.Cu at (17.9, 190.6)
- added C701: 100n, Capacitor_SMD:C_0402_1005Metric, F.Cu at (-33.4, 111.5)
- added C702: 100n, Capacitor_SMD:C_0402_1005Metric, F.Cu at (-32.6, 116.2)
- added C703: 100n, Capacitor_SMD:C_0402_1005Metric, F.Cu at (-32.6, 118.2)
- added C704: 100n, Capacitor_SMD:C_0402_1005Metric, F.Cu at (-30.5, 111.5)
- added C705: 100n, Capacitor_SMD:C_0402_1005Metric, F.Cu at (-29.7, 116.2)
- added C706: 100n, Capacitor_SMD:C_0402_1005Metric, F.Cu at (-29.7, 118.2)
- added C707: 100n, Capacitor_SMD:C_0402_1005Metric, F.Cu at (-27.6, 111.5)
- added C708: 100n, Capacitor_SMD:C_0402_1005Metric, F.Cu at (-26.8, 116.2)
- added C709: 100n, Capacitor_SMD:C_0402_1005Metric, F.Cu at (-26.8, 118.2)
- added C801: 100n, Capacitor_SMD:C_0402_1005Metric, F.Cu at (-164.9, 188.7)
- added C802: 100n, Capacitor_SMD:C_0402_1005Metric, F.Cu at (-164.9, 190.6)
- added REF**: Keyboard v2, keyboard_footprints:Keyboard v2, F.Cu at (300.0, 130.0)
- added REF**: Keyboard v2, keyboard_footprints:Keyboard v2, B.Cu at (145.0, 130.0)
- C1303, C1304, C1305, C1306, C1309, C1310, C1311, C1312, C1313, C1314, C1316, C1317, C1321, C1322, C803, C804, C805, C806, C809, C810, C811, C812, C813, C814, C816, C817, C821, C822: footprint Capacitor_SMD:C_0201_0603Metric -> Capacitor_SMD:C_0402_1005Metric
- D1201, D1202, D1203, D1204, D1205, D1206, D1207, D1208, D1209, D1210, D1211, D1212, D1213, D1214, D1215, D1216, D1217, D1218, D1219, D1220, D1221, D1222, D1223, D1224, D1225, D1226, D1227, D701, D702, D703, D704, D705, D706, D707, D708, D709, D710, D711, D712, D713, D714, D715, D716, D717, D718, D719, D720, D721, D722, D723, D724, D725, D726, D727: moved to B.Cu
- J201: footprint keyboard_parts:debug_header -> keyboard_footprints:debug_header; moved to F.Cu
- J301: footprint keyboard_parts:debug_header -> keyboard_footprints:debug_header
- moved J602 447.4 mm to (336.0, 79.2), turned to 180 degrees
- moved SW721 440.5 mm to (338.0, 100.0)
- moved SW722 440.2 mm to (338.0, 119.0)
- moved SW728 439.8 mm to (357.0, 157.0)
- moved SW727 439.7 mm to (357.0, 138.0)
- moved SW726 439.6 mm to (357.0, 119.0)
- moved SW725 439.5 mm to (357.0, 100.0)
- moved D703 434.8 mm to (356.2, 152.2), turned to 180 degrees
- moved SW724 428.1 mm to (338.0, 157.0)
- moved SW702 427.6 mm to (273.6, 180.3), turned to 30 degrees
- moved SW723 427.5 mm to (338.0, 138.0)
- moved J601 427.4 mm to (318.0, 79.2), turned to 180 degrees
- moved SW708 421.9 mm to (281.0, 99.0)
- moved SW720 420.5 mm to (319.0, 153.0)
- moved SW719 420.3 mm to (319.0, 134.0)
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Connections:
- C1311 pad 1: +1V8 -> +3V3
- C813 pad 1: +3V3 -> +1V8
- C816 pad 1: +1V8 -> +3V3
- C817 pad 1: +1V8 -> +3V3
- U1301 pad B11: unconnected-(U1301A-PA14-PadB11) -> /Left/Main MCU Left/SWCLK
- U1301 pad C10: unconnected-(U1301A-PA13-PadC10) -> /Left/Main MCU Left/SWDIO
- U1301 pad C11: unconnected-(U1301A-PA12-PadC11) -> /Left/USB/USB3_DP
- U1301 pad C12: unconnected-(U1301A-PA11-PadC12) -> /Left/USB/USB3_DN
- U1301 pad C5: unconnected-(U1301A-PB7-PadC5) -> /Left/Display/DSI_TE
- U801 pad B11: unconnected-(U801A-PA14-PadB11) -> /Right/Main MCU Right/SWCLK
- U801 pad C10: unconnected-(U801A-PA13-PadC10) -> /Right/Main MCU Right/SWDIO
- U801 pad C11: unconnected-(U801A-PA12-PadC11) -> /Right/USB/USB3_DP
- U801 pad C12: unconnected-(U801A-PA11-PadC12) -> /Right/USB/USB3_DN
- U801 pad C5: unconnected-(U801A-PB7-PadC5) -> /Right/Display/DSI_TE
Other:
- board size 143.8 x 139.6 mm -> 283.4 x 102.2 mm

Commit message: Started routing
Parts:
- AE202, AE302, IC1401, IC501, J1101, J201, J301, J401, SW1402, SW502, TP1401, TP1402, TP501, TP502, U1001, U1101, U1301, U1504, U1505, U401, U604, U605, U801, U901: moved to B.Cu
- moved AE302 443.8 mm to (284.1, 88.1), turned to 180 degrees
- moved U801 404.6 mm to (247.0, 125.4), turned to 180 degrees
- moved J301 391.4 mm to (245.1, 112.6), turned to -150 degrees
- moved SW502 389.5 mm to (279.0, 169.0), turned to -90 degrees
- moved TP502 372.3 mm to (253.0, 167.0), turned to -90 degrees
- moved U604 371.7 mm to (331.0, 88.8), turned to 180 degrees
- moved U901 369.4 mm to (290.0, 105.0), turned to 180 degrees
- moved TP501 366.7 mm to (247.9, 167.0), turned to -90 degrees
- moved IC501 362.7 mm to (255.2, 174.0), turned to 180 degrees
- moved U605 354.9 mm to (340.8, 89.0), turned to 180 degrees
- moved J201 343.5 mm to (199.9, 112.6), turned to 150 degrees
- moved J401 341.6 mm to (237.0, 126.5), turned to 90 degrees
- moved U401 337.1 mm to (232.8, 117.2), turned to 180 degrees
- moved TP1401 313.5 mm to (196.2, 167.0), turned to 90 degrees
- moved AE202 313.3 mm to (160.9, 88.1), turned to 180 degrees
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