File: PCBs/keyboard_v2/display.kicad_sch (KiCad schematic)
At the start: 11 parts, among them U401 RT4730WSC

Commit message: V2 progress
Parts:
- renumbered C401 to C1101, C402 to C1102, C403 to C1103, C404 to C1104, C405 to C1105, C406 to C1106, C407 to C1107, C408 to C1108, C409 to C1109, L401 to L1101, U401 to U1101
Changed lines of the file:
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@@
 		(on_board yes)
 		(dnp no)
-		(property "Reference" "C406"
+		(property "Reference" "C1106"
 			(at 147.32 115.5763 0)
 			(effects
@@
 		(on_board yes)
 		(dnp no)
-		(property "Reference" "L401"
+		(property "Reference" "L1101"
 			(at 125.73 80.645 0)
 			(effects
@@
 		(on_board yes)
 		(dnp no)
-		(property "Reference" "C401"
+		(property "Reference" "C1101"
 			(at 60.96 80.0163 0)
 			(effects
@@
 		(on_board yes)
 		(dnp no)
-		(property "Reference" "C409"
+		(property "Reference" "C1109"
 			(at 177.8 115.5763 0)
 			(effects
@@
 		(on_board yes)
 		(dnp no)
-		(property "Reference" "C405"
+		(property "Reference" "C1105"
 			(at 137.16 115.5763 0)
 			(effects
@@
 		(dnp no)
 		(fields_autoplaced yes)
-		(property "Reference" "#PWR0403"
+		(property "Reference" "#PWR01103"
 			(at 175.26 135.89 0)
 			(effects
@@
 		(dnp no)
 		(fields_autoplaced yes)
-		(property "Reference" "#PWR0401"
+		(property "Reference" "#PWR01101"
 			(at 63.5 77.47 0)
 			(effects
@@
 		(on_board yes)
 		(dnp no)
-		(property "Reference" "C404"
+		(property "Reference" "C1104"
 			(at 127 115.5763 0)
 			(effects
@@
 		(on_board yes)
 		(dnp no)
-		(property "Reference" "C407"
+		(property "Reference" "C1107"
 			(at 157.48 115.5763 0)
 			(effects
@@
 		(on_board yes)
 		(dnp no)
-		(property "Reference" "C403"
+		(property "Reference" "C1103"
 			(at 76.2 102.8763 0)
 			(effects
@@
 		(dnp no)
 		(fields_autoplaced yes)
-		(property "Reference" "#PWR0402"
+		(property "Reference" "#PWR01102"
 			(at 63.5 95.25 0)
 			(effects
@@
 		(on_board yes)
 		(dnp no)
-		(property "Reference" "U401"
+		(property "Reference" "U1101"
 			(at 101.6 68.58 0)
 			(effects
@@
 		(on_board yes)
 		(dnp no)
-		(property "Reference" "C402"
+		(property "Reference" "C1102"
 			(at 73.66 80.0163 0)
 			(effects
@@
 		(on_board yes)
 		(dnp no)
-		(property "Reference" "C408"
+		(property "Reference" "C1108"
 			(at 167.64 115.5763 0)
 			(effects

Commit message: V2 Progress
Parts:
- added J1101: FH26W-27S-0.3SHW_60_, keyboard_footprints:FH26W27S03SHW60, symbol FH26W-27S-0_3SHW_60_:FH26W-27S-0.3SHW_60_
Changed lines of the file:
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@@
+		)
+	)
+	(hierarchical_label "DSI_CKN"
+		(shape input)
+		(at 165.1 38.1 0)
+		(fields_autoplaced yes)
+		(effects
+			(font
+				(size 1.27 1.27)
+			)
+			(justify left)
+		)
+	)
+	(hierarchical_label "DSI_TE"
+		(shape output)
+		(at 165.1 33.02 0)
+		(fields_autoplaced yes)
+		(effects
+			(font
+				(size 1.27 1.27)
+			)
+			(justify left)
+		)
+	)
+	(hierarchical_label "DSI_D0N"
+		(shape bidirectional)
+		(at 165.1 43.18 0)
+		(fields_autoplaced yes)
+		(effects
+			(font
+				(size 1.27 1.27)
+			)
+			(justify left)
+		)
+	)
+	(hierarchical_label "DSI_CKP"
+		(shape input)
+		(at 165.1 35.56 0)
+		(fields_autoplaced yes)
+		(effects
+			(font
+				(size 1.27 1.27)
+			)
+			(justify left)
+		)
+	)
+	(hierarchical_label "DSI_D0P"
+		(shape bidirectional)
+		(at 165.1 40.64 0)
+		(fields_autoplaced yes)
+		(effects
+			(font
+				(size 1.27 1.27)
+			)
+			(justify left)
 		)
 	)
@@
 					(unit 1)
 				)
+			)
+		)
+	)
+	(symbol
+		(lib_id "FH26W-27S-0_3SHW_60_:FH26W-27S-0.3SHW_60_")
+		(at 241.3 55.88 0)
+		(unit 1)
+		(exclude_from_sim no)
+		(in_bom yes)
+		(on_board yes)
+		(dnp no)
+		(fields_autoplaced yes)
+		(property "Reference" "J1101"
+			(at 241.3 50.8 0)
+			(effects
+				(font
+					(size 1.27 1.27)
+				)
+			)
+		)
+		(property "Value" "FH26W-27S-0.3SHW_60_"
+			(at 241.3 53.34 0)
+			(effects
+				(font
+					(size 1.27 1.27)
+				)
+			)
+		)
+		(property "Footprint" "keyboard_footprints:FH26W27S03SHW60"
+			(at 223.52 132.08 0)
+			(effects
+				(font
+					(size 1.27 1.27)
+				)
+				(justify left top)
+				(hide yes)
+			)
+		)
+		(property "Datasheet" "https://www.hirose.com/product/document?clcode=CL0580-2400-9-60&productname=FH26W-27S-0.3SHW(60)&series=FH26&documenttype=2DDrawing&lang=en&documentid=0001001683"
+			(at 285.75 245.72 0)
+			(effects
+				(font
+					(size 1.27 1.27)
+				)
+				(justify left top)
+				(hide yes)
+			)
+		)
+		(property "Description" "FFC & FPC Connectors"
+			(at 241.3 129.54 0)
+			(effects
+				(font
+					(size 1.27 1.27)
+				)
+				(hide yes)
+			)
+		)
+		(property "Height" "2.3"
+			(at 285.75 445.72 0)
+			(effects
+				(font
+					(size 1.27 1.27)
+				)
+				(justify left top)
+				(hide yes)
+			)
+		)
+		(property "Mouser Part Number" "798-FH26W27S03SHW60"
+			(at 285.75 545.72 0)
+			(effects
+				(font
+					(size 1.27 1.27)
+				)
+				(justify left top)
+				(hide yes)
+			)
+		)
+		(property "Mouser Price/Stock" "https://www.mouser.co.uk/ProductDetail/Hirose-Connector/FH26W-27S-0.3SHW60?qs=vcbW%252B4%252BSTIouYwvbDemSLQ%3D%3D"
+			(at 285.75 645.72 0)
+			(effects
+				(font
+					(size 1.27 1.27)
+				)
+				(justify left top)
+				(hide yes)
+			)
+		)
+		(property "Manufacturer_Name" "Hirose"
+			(at 285.75 745.72 0)
+			(effects
+				(font
+					(size 1.27 1.27)
+				)
+				(justify left top)
+				(hide yes)
+			)
+		)
+		(property "Manufacturer_Part_Number" "FH26W-27S-0.3SHW(60)"
+			(at 285.75 845.72 0)
+			(effects
+				(font
+					(size 1.27 1.27)
+				)
+				(justify left top)
+				(hide yes)
+			)
+		)
+		(pin "23"
+		)
+		(pin "18"
+		)
+		(pin "6"
+		)
+		(pin "24"
+		)
+		(pin "MP2"
+		)
+		(pin "16"
+		)
+		(pin "2"
+		)
+		(pin "20"
+		)
+		(pin "12"
+		)
+		(pin "4"
+		)
+		(pin "15"
+		)
+		(pin "17"
+		)
+		(pin "13"
+		)
+		(pin "26"
+		)
+		(pin "5"
+		)
+		(pin "21"
+		)
+		(pin "25"
+		)
+		(pin "22"
+		)
+		(pin "11"
+		)
+		(pin "10"
+		)
+		(pin "1"
+		)
+		(pin "27"
+		)
+		(pin "14"
+		)
+		(pin "7"
+		)
+		(pin "9"
+		)
+		(pin "3"
+		)
+		(pin "8"
+		)
+		(pin "MP1"
+		)
+		(pin "19"
+		)
+		(instances
+			(project "keyboard_v2"
+				(path "/e2360b7f-be71-48d9-b398-9f8cd45479d6/8d5749a2-4d36-4f17-8c57-9c8b87d773d6/477316a5-f8d9-40b1-a704-da1d199f3a0b"
+					(reference "J1101")
+					(unit 1)
+				)
+				(path "/e2360b7f-be71-48d9-b398-9f8cd45479d6/b599252a-0e44-4760-9c79-385d4380db60/8fed583c-0d52-4b53-b8a4-fd3365ae1417"
+					(reference "J401")
+					(unit 1)
+				)

Commit message: Display schematic done
Connections:
- net AVDD: now also J1101.4
- net DSI_CKN: now also J1101.11
- net DSI_CKP: now also J1101.10
- net DSI_D0N: now also J1101.8
- net DSI_D0P: now also J1101.7
- net DSI_TE: now also J1101.20
- net ELVDD: now also J1101.2
- net ELVSS: now also J1101.1
- net GND: now also J1101.12, J1101.14, J1101.15, J1101.18, J1101.22, J1101.6, J1101.9, J1101.MP1, J1101.MP2
- net SWIRE: now also J1101.21
- net IM0: now reaches J1101.16
- net +1V8: now reaches J1101.17
- net +1V8: now also J1101.5
- net RST_DISP: now reaches J1101.19
- net +3V3: now reaches J1101.23
- net RST_TP: now reaches J1101.24
- net INT_TP: now reaches J1101.25
- net SCL_TP: now reaches J1101.26
- net SDA_TP: now reaches J1101.27
- no-connect marks 0 -> 2
Other:
- note added: "CS"
- note added: "DCX"
- note added: "GND"
- note added: "MTP"
- note added: "SCL"
- note added: "SDA"
- note added: "SDO"
- note added: "VDDIO"
- note added: "VDD_TP"
