File: PCBs/keyboard_v2/left.kicad_sch (KiCad schematic)
At the start: 0 parts

Commit message: V2 Progress
Other:
- sheet Bluetooth ports: added RST, SWCLK, SWDIO, UART_RX, UART_TX; removed none
- sheet Display ports: added AVDDEN, DSI_CKN, DSI_CKP, DSI_D0N, DSI_D0P, DSI_TE; removed none
- sheet Keys Left ports: added ENC_A, ENC_B, ENC_SW, KEY_A1, KEY_A2, KEY_A3, KEY_A4, KEY_A5, KEY_A6, KEY_B1, KEY_B2, KEY_B3, KEY_B4, KEY_B5, KEY_B6, KEY_C1, KEY_C2, KEY_C3, KEY_C4, KEY_C5, KEY_C6, KEY_D1, KEY_D2, KEY_D3, KEY_D4, KEY_D5, KEY_D6, KEY_E1, KEY_E2, KEY_E3, LED1; removed none
- sheet Main MCU Left ports: added DSI_CKN, DSI_CKP, DSI_D0N, DSI_D0P, DSI_TE, ENC_A, ENC_B, ENC_SW, KEY_A1, KEY_A2, KEY_A3, KEY_A4, KEY_A5, KEY_A6, KEY_B1, KEY_B2, KEY_B3, KEY_B4, KEY_B5, KEY_B6, KEY_C1, KEY_C2, KEY_C3, KEY_C4, KEY_C5, KEY_C6, KEY_D1, KEY_D2, KEY_D3, KEY_D4, KEY_D5, KEY_D6, KEY_E1, KEY_E2, KEY_E3, NEOPIXEL, RST, SWCLK, SWDIO, USB_DN, USB_DP; removed none
- sheet Power ports: added +1V8, +3V3, +VBAT, +VSYS, BTN, ENCHG, INT, ISYS, SCL, SDA; removed none
- sheet USB ports: added RST, SCL, SDA, SWCLK, SWDIO, UART_RX, UART_TX, USB_DN, USB_DP; removed none

Commit message: Display schematic done
Other:
- sheet Display ports: added IM0, INT_TP, RST_DISP, RST_TP, SCL_TP, SDA_TP; removed none
- sheet USB ports: added none; removed SCL, SDA

Commit message: V2 Schematic mostly done
Parts:
- added AE202: Antenna_Shield, RF_Antenna:Texas_SWRA117D_2.4GHz_Left, symbol Device:Antenna_Shield
- added J201: TMS-115-01-G-S, keyboard_parts:debug_header, symbol Connector_Generic:Conn_01x15
Connections:
- net Bluetooth/RST: now also J201.11 (Pin_11)
- net Bluetooth/SWCLK: now also J201.13 (Pin_13)
- net Bluetooth/SWDIO: now also J201.12 (Pin_12)
- net Main MCU Left/RST: now also J201.1 (Pin_1)
- net Main MCU Left/SWCLK: now also J201.3 (Pin_3)
- net Main MCU Left/SWDIO: now also J201.2 (Pin_2)
- net USB/SWCLK: now also J201.8 (Pin_8)
- net USB/SWDIO: now also J201.7 (Pin_7)
- new net +1V8: J201.15 (Pin_15), J201.5 (Pin_5)
- new net +3V3: J201.10 (Pin_10)
- new net Bluetooth/ANT: AE202.1 (A)
- new net GND: AE202.2 (Shield), J201.14 (Pin_14), J201.4 (Pin_4), J201.9 (Pin_9)
- new net Main MCU Left/USB_RST: J201.6 (Pin_6)
Other:
- sheet Bluetooth ports: added ANT; removed none
- sheet Keys Left ports: added NEOPIXEL; removed LED1
- sheet Main MCU Left ports: added AVDDEN, BLE_RST, BLE_UART_RX, BLE_UART_TX, IM0, INT_TP, ISYS, PWR_ENCHG, PWR_INT, PWR_MR, PWR_SCL, PWR_SDA, RST_DISP, RST_TP, SCL_TP, SDA_TP, USB_RST, USB_UART_RX, USB_UART_TX; removed none
- sheet Power ports: added MR; removed +1V8, +3V3, +VBAT, +VSYS, BTN

Commit message: Added debug header footprint
Parts:
- J201: footprint keyboard_parts:debug_header -> keyboard_footprints:debug_header
Changed lines of the file:
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@@
 			)
 		)
-		(property "Footprint" "keyboard_parts:debug_header"
+		(property "Footprint" "keyboard_footprints:debug_header"
 			(at 116.84 33.02 0)
 			(effects

Commit message: Layout in progress
Parts:
- removed AE202: Antenna_Shield, RF_Antenna:Texas_SWRA117D_2.4GHz_Left, symbol Device:Antenna_Shield
- added ANT201: ANT3216A063R2400A, keyboard_footprints:ANTC3016X65N, symbol ANT3216A063R2400A:ANT3216A063R2400A
Connections:
- net Bluetooth/ANT: now also ANT201.2 (FEED2)
- net GND: now also ANT201.1 (FEED1), ANT201.3 (GND)
Other:
- sheet Keys Left renamed Keys
- sheet Main MCU Left renamed Main MCU
- sheet USB: file usb.kicad_sch -> usb_left.kicad_sch
Changed lines of the file:
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@@
+	)
+	(junction
+		(at 55.88 53.34)
+		(diameter 0)
+		(color 0 0 0 0)
 	)
 	(junction
@@
 	(wire
 		(pts
+			(xy 55.88 53.34) (xy 55.88 55.88)
+		)
+		(stroke
+			(width 0)
+			(type default)
+		)
+	)
+	(wire
+		(pts
 			(xy 91.44 60.96) (xy 142.24 60.96)
 		)
@@
 	(wire
 		(pts
-			(xy 60.96 48.26) (xy 60.96 50.8)
-		)
-		(stroke
-			(width 0)
-			(type default)
-		)
-	)
-	(wire
-		(pts
 			(xy 124.46 50.8) (xy 124.46 38.1)
 		)
@@
 	(wire
 		(pts
+			(xy 55.88 48.26) (xy 55.88 53.34)
+		)
+		(stroke
+			(width 0)
+			(type default)
+		)
+	)
+	(wire
+		(pts
 			(xy 121.92 81.28) (xy 91.44 81.28)
 		)
@@
 	(wire
 		(pts
-			(xy 63.5 50.8) (xy 66.04 50.8)
-		)
-		(stroke
-			(width 0)
-			(type default)
-		)
-	)
-	(wire
-		(pts
 			(xy 114.3 40.64) (xy 114.3 38.1)
 		)
@@
 	(wire
 		(pts
-			(xy 63.5 48.26) (xy 63.5 50.8)
-		)
-		(stroke
-			(width 0)
-			(type default)
-		)
-	)
-	(wire
-		(pts
 			(xy 167.64 45.72) (xy 193.04 45.72)
 		)
@@
 	(wire
 		(pts
+			(xy 53.34 53.34) (xy 55.88 53.34)
+		)
+		(stroke
+			(width 0)
+			(type default)
+		)
+	)
+	(wire
+		(pts
 			(xy 91.44 142.24) (xy 142.24 142.24)
 		)
@@
 	(wire
 		(pts
+			(xy 53.34 48.26) (xy 55.88 48.26)
+		)
+		(stroke
+			(width 0)
+			(type default)
+		)
+	)
+	(wire
+		(pts
 			(xy 167.64 111.76) (xy 193.04 111.76)
 		)
@@
 		(pts
 			(xy 91.44 55.88) (xy 109.22 55.88)
+		)
+		(stroke
+			(width 0)
+			(type default)
+		)
+	)
+	(wire
+		(pts
+			(xy 53.34 50.8) (xy 66.04 50.8)
 		)
 		(stroke
@@
 	)
 	(symbol
+		(lib_id "ANT3216A063R2400A:ANT3216A063R2400A")
+		(at 53.34 48.26 0)
+		(mirror y)
+		(unit 1)
+		(exclude_from_sim no)
+		(in_bom yes)
+		(on_board yes)
+		(dnp no)
+		(fields_autoplaced yes)
+		(property "Reference" "ANT201"
+			(at 41.91 40.64 0)
+			(effects
+				(font
+					(size 1.27 1.27)
+				)
+			)
+		)
+		(property "Value" "ANT3216A063R2400A"
+			(at 41.91 43.18 0)
+			(effects
+				(font
+					(size 1.27 1.27)
+				)
+			)
+		)
+		(property "Footprint" "keyboard_footprints:ANTC3016X65N"
+			(at 34.29 143.18 0)
+			(effects
+				(font
+					(size 1.27 1.27)
+				)
+				(justify left top)
+				(hide yes)
+			)
+		)
+		(property "Datasheet" "https://media.digikey.com/pdf/Data%20Sheets/Yageo%20PDFs/ANT3216A063R2400A_Rev2014.pdf"
+			(at 34.29 243.18 0)
+			(effects
+				(font
+					(size 1.27 1.27)
+				)
+				(justify left top)
+				(hide yes)
+			)
+		)
+		(property "Description" "Antennas 1W, 2.45GHz, 3216"
+			(at 53.34 63.5 0)
+			(effects
+				(font
+					(size 1.27 1.27)
+				)
+				(hide yes)
+			)
+		)
+		(property "Height" "0.65"
+			(at 34.29 443.18 0)
+			(effects
+				(font
+					(size 1.27 1.27)
+				)
+				(justify left top)
+				(hide yes)
+			)
+		)
+		(property "Mouser Part Number" "603-ANT3216A063R2400"
+			(at 34.29 543.18 0)
+			(effects
+				(font
+					(size 1.27 1.27)
+				)
+				(justify left top)
+				(hide yes)
+			)
+		)
+		(property "Mouser Price/Stock" "https://www.mouser.co.uk/ProductDetail/Pulse-Electronics/ANT3216A063R2400A?qs=CqAAFKzD4h%252BYK9SO0hbvNw%3D%3D"
+			(at 34.29 643.18 0)
+			(effects
+				(font
+					(size 1.27 1.27)
+				)
+				(justify left top)
+				(hide yes)
+			)
+		)
+		(property "Manufacturer_Name" "Pulse Electronics"
+			(at 34.29 743.18 0)
+			(effects
+				(font
+					(size 1.27 1.27)
+				)
+				(justify left top)
+				(hide yes)
+			)
+		)
+		(property "Manufacturer_Part_Number" "ANT3216A063R2400A"
+			(at 34.29 843.18 0)
+			(effects
+				(font
+					(size 1.27 1.27)
+				)
+				(justify left top)
+				(hide yes)
+			)
+		)
+		(pin "1"
+		)
+		(pin "2"
+		)
+		(pin "3"
+		)
+		(instances
+			(project ""
+				(path "/e2360b7f-be71-48d9-b398-9f8cd45479d6/8d5749a2-4d36-4f17-8c57-9c8b87d773d6"
+					(reference "ANT201")
+					(unit 1)
+				)
+			)
+		)
+	)
+	(symbol
 		(lib_id "power:+1V8")
 		(at 93.98 38.1 0)
@@
 	)
 	(symbol
-		(lib_id "Device:Antenna_Shield")
-		(at 63.5 43.18 0)
-		(mirror y)
-		(unit 1)
-		(exclude_from_sim no)
-		(in_bom yes)
-		(on_board yes)
-		(dnp no)
-		(property "Reference" "AE202"
-			(at 59.69 41.2749 0)
-			(effects
-				(font
-					(size 1.27 1.27)
-				)
-				(justify left)
-			)
-		)
-		(property "Value" "Antenna_Shield"
-			(at 59.69 43.8149 0)
-			(effects
-				(font
-					(size 1.27 1.27)
-				)
-				(justify left)
-			)
-		)
-		(property "Footprint" "RF_Antenna:Texas_SWRA117D_2.4GHz_Left"
-			(at 63.5 40.64 0)
-			(effects
-				(font
-					(size 1.27 1.27)
-				)
-				(hide yes)
-			)
-		)
-		(property "Datasheet" "~"
-			(at 63.5 40.64 0)
-			(effects
-				(font
-					(size 1.27 1.27)
-				)
-				(hide yes)
-			)
-		)
-		(property "Description" "Antenna with extra pin for shielding"
-			(at 63.5 43.18 0)
-			(effects
-				(font
-					(size 1.27 1.27)
-				)
-				(hide yes)
-			)
-		)
-		(pin "1"
-		)
-		(pin "2"
-		)
-		(instances
-			(project ""
-				(path "/e2360b7f-be71-48d9-b398-9f8cd45479d6/8d5749a2-4d36-4f17-8c57-9c8b87d773d6"
-					(reference "AE202")
-					(unit 1)
-				)
-			)
-		)
-	)
-	(symbol
 		(lib_id "Connector_Generic:Conn_01x15")
 		(at 116.84 33.02 270)
@@
 	(symbol
 		(lib_id "power:GND")
-		(at 60.96 50.8 0)
+		(at 55.88 55.88 0)
 		(unit 1)
 		(exclude_from_sim no)
@@
 		(fields_autoplaced yes)
 		(property "Reference" "#PWR0205"
-			(at 60.96 57.15 0)
+			(at 55.88 62.23 0)
 			(effects
 				(font
@@
 		)
 		(property "Value" "GND"
-			(at 60.96 55.88 0)
+			(at 55.88 60.96 0)
 			(effects
 				(font
@@
 		)
 		(property "Footprint" ""
-			(at 60.96 50.8 0)
+			(at 55.88 55.88 0)
 			(effects
 				(font
@@
 		)
 		(property "Datasheet" ""
-			(at 60.96 50.8 0)
+			(at 55.88 55.88 0)
 			(effects
 				(font
@@
 		)
 		(property "Description" "Power symbol creates a global label with name \"GND\" , ground"
-			(at 60.96 50.8 0)
+			(at 55.88 55.88 0)
 			(effects
 				(font
@@
 		)
 		(instances
-			(project ""
+			(project "keyboard_v2"
 				(path "/e2360b7f-be71-48d9-b398-9f8cd45479d6/8d5749a2-4d36-4f17-8c57-9c8b87d773d6"
 					(reference "#PWR0205")
@@
 			)
 		)
-		(property "Sheetfile" "usb.kicad_sch"
+		(property "Sheetfile" "usb_left.kicad_sch"
 			(at 66.04 99.6446 0)
 			(effects
@@
 			(color 0 0 0 0.0000)
 		)
-		(property "Sheetname" "Keys Left"
+		(property "Sheetname" "Keys"
 			(at 193.04 42.4684 0)
 			(effects
@@
 			)
 		)
-		(pin "ANT" output
+		(pin "ANT" bidirectional
 			(at 66.04 50.8 180)
 			(effects
@@
 			(color 0 0 0 0.0000)
 		)
-		(property "Sheetname" "Main MCU Left"
+		(property "Sheetname" "Main MCU"
 			(at 142.24 42.4684 0)
 			(effects
