File: PCBs/keyboard_v2/right.kicad_sch (KiCad schematic)
At the start: 0 parts

Commit message: V2 progress
Other:
- sheet Bluetooth ports: added RST, SWCLK, SWDIO, UART_RX, UART_TX; removed none
- sheet Display ports: added AVDDEN; removed none
- sheet Keys Right ports: added ENC_A, ENC_B, ENC_SW, KEY_A10, KEY_A11, KEY_A12, KEY_A7, KEY_A8, KEY_A9, KEY_B10, KEY_B11, KEY_B12, KEY_B7, KEY_B8, KEY_B9, KEY_C10, KEY_C11, KEY_C12, KEY_C7, KEY_C8, KEY_C9, KEY_D10, KEY_D11, KEY_D12, KEY_D7, KEY_D8, KEY_D9, KEY_E4, KEY_E5, KEY_E6, LED1; removed none
- sheet Main MCU Right ports: added ENC_A, ENC_B, ENC_SW, KEY_A10, KEY_A11, KEY_A12, KEY_A7, KEY_A8, KEY_A9, KEY_B10, KEY_B11, KEY_B12, KEY_B7, KEY_B8, KEY_B9, KEY_C10, KEY_C11, KEY_C12, KEY_C7, KEY_C8, KEY_C9, KEY_D10, KEY_D11, KEY_D12, KEY_D7, KEY_D8, KEY_D9, KEY_E4, KEY_E5, KEY_E6, NEOPIXEL, RST, SWCLK, SWDIO; removed none
- sheet Power ports: added +1V8, +3V3, +VBAT, +VSYS, BTN, ENCHG, INT, ISYS, SCL, SDA; removed none
- sheet USB ports: added RST, SCL, SDA, SWCLK, SWDIO, UART_RX, UART_TX; removed none

Commit message: V2 Progress
Other:
- sheet Display ports: added DSI_CKN, DSI_CKP, DSI_D0N, DSI_D0P, DSI_TE; removed none
- sheet Main MCU Right ports: added DSI_CKN, DSI_CKP, DSI_D0N, DSI_D0P, DSI_TE, USB_DN, USB_DP; removed none
- sheet USB ports: added USB_DN, USB_DP; removed none

Commit message: Display schematic done
Other:
- sheet Display ports: added IM0, INT_TP, RST_DISP, RST_TP, SCL_TP, SDA_TP; removed none
- sheet USB ports: added none; removed SCL, SDA

Commit message: V2 Schematic mostly done
Parts:
- added AE302: Antenna_Shield, RF_Antenna:Texas_SWRA117D_2.4GHz_Right, symbol Device:Antenna_Shield
- added J301: TMS-115-01-G-S, keyboard_parts:debug_header, symbol Connector_Generic:Conn_01x15
Connections:
- net Bluetooth/RST: now also J301.5 (Pin_5)
- net Bluetooth/SWCLK: now also J301.3 (Pin_3)
- net Bluetooth/SWDIO: now also J301.4 (Pin_4)
- net Main MCU Right/RST: now also J301.15 (Pin_15)
- net Main MCU Right/SWCLK: now also J301.13 (Pin_13)
- net Main MCU Right/SWDIO: now also J301.14 (Pin_14)
- net USB/SWCLK: now also J301.8 (Pin_8)
- net USB/SWDIO: now also J301.9 (Pin_9)
- new net +1V8: J301.1 (Pin_1), J301.11 (Pin_11)
- new net +3V3: J301.6 (Pin_6)
- new net Bluetooth/ANT: AE302.1 (A)
- new net GND: AE302.2 (Shield), J301.12 (Pin_12), J301.2 (Pin_2), J301.7 (Pin_7)
- new net Main MCU Right/USB_RST: J301.10 (Pin_10)
Other:
- sheet Bluetooth ports: added ANT; removed none
- sheet Keys Right ports: added NEOPIXEL; removed LED1
- sheet Main MCU Right ports: added AVDDEN, BLE_RST, BLE_UART_RX, BLE_UART_TX, IM0, INT_TP, ISYS, PWR_ENCHG, PWR_INT, PWR_MR, PWR_SCL, PWR_SDA, RST_DISP, RST_TP, SCL_TP, SDA_TP, USB_RST, USB_UART_RX, USB_UART_TX; removed none
- sheet Power ports: added MR; removed +1V8, +3V3, +VBAT, +VSYS, BTN

Commit message: Added debug header footprint
Parts:
- J301: footprint keyboard_parts:debug_header -> keyboard_footprints:debug_header
Changed lines of the file:
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@@
 			)
 		)
-		(property "Footprint" "keyboard_parts:debug_header"
+		(property "Footprint" "keyboard_footprints:debug_header"
 			(at 119.38 30.48 0)
 			(effects

Commit message: Layout in progress
Parts:
- removed AE302: Antenna_Shield, RF_Antenna:Texas_SWRA117D_2.4GHz_Right, symbol Device:Antenna_Shield
- added ANT301: ANT3216A063R2400A, keyboard_footprints:ANTC3016X65N, symbol ANT3216A063R2400A:ANT3216A063R2400A
Connections:
- net Bluetooth/ANT: now also ANT301.1 (FEED1)
- net GND: now also ANT301.2 (FEED2), ANT301.3 (GND)
Other:
- sheet Keys Right renamed Keys
- sheet Main MCU Right renamed Main MCU
- sheet USB: file usb.kicad_sch -> usb_right.kicad_sch
Changed lines of the file:
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@@
+	)
+	(junction
+		(at 58.42 53.34)
+		(diameter 0)
+		(color 0 0 0 0)
 	)
 	(junction
@@
 	(wire
 		(pts
+			(xy 58.42 53.34) (xy 58.42 55.88)
+		)
+		(stroke
+			(width 0)
+			(type default)
+		)
+	)
+	(wire
+		(pts
 			(xy 170.18 78.74) (xy 195.58 78.74)
 		)
@@
 	(wire
 		(pts
-			(xy 66.04 48.26) (xy 68.58 48.26)
-		)
-		(stroke
-			(width 0)
-			(type default)
-		)
-	)
-	(wire
-		(pts
 			(xy 170.18 96.52) (xy 195.58 96.52)
 		)
@@
 	(wire
 		(pts
+			(xy 55.88 48.26) (xy 68.58 48.26)
+		)
+		(stroke
+			(width 0)
+			(type default)
+		)
+	)
+	(wire
+		(pts
 			(xy 104.14 38.1) (xy 116.84 38.1)
 		)
@@
 	(wire
 		(pts
-			(xy 66.04 45.72) (xy 66.04 48.26)
+			(xy 55.88 50.8) (xy 58.42 50.8)
 		)
 		(stroke
@@
 	(wire
 		(pts
+			(xy 55.88 53.34) (xy 58.42 53.34)
+		)
+		(stroke
+			(width 0)
+			(type default)
+		)
+	)
+	(wire
+		(pts
 			(xy 93.98 114.3) (xy 144.78 114.3)
 		)
@@
 	(wire
 		(pts
+			(xy 58.42 50.8) (xy 58.42 53.34)
+		)
+		(stroke
+			(width 0)
+			(type default)
+		)
+	)
+	(wire
+		(pts
 			(xy 170.18 132.08) (xy 195.58 132.08)
 		)
@@
 		(pts
 			(xy 129.54 48.26) (xy 129.54 45.72)
-		)
-		(stroke
-			(width 0)
-			(type default)
-		)
-	)
-	(wire
-		(pts
-			(xy 63.5 45.72) (xy 63.5 48.26)
 		)
 		(stroke
@@
 	)
 	(symbol
-		(lib_id "Device:Antenna_Shield")
-		(at 66.04 40.64 0)
+		(lib_id "power:GND")
+		(at 58.42 55.88 0)
+		(unit 1)
+		(exclude_from_sim no)
+		(in_bom yes)
+		(on_board yes)
+		(dnp no)
+		(fields_autoplaced yes)
+		(property "Reference" "#PWR0305"
+			(at 58.42 62.23 0)
+			(effects
+				(font
+					(size 1.27 1.27)
+				)
+				(hide yes)
+			)
+		)
+		(property "Value" "GND"
+			(at 58.42 60.96 0)
+			(effects
+				(font
+					(size 1.27 1.27)
+				)
+			)
+		)
+		(property "Footprint" ""
+			(at 58.42 55.88 0)
+			(effects
+				(font
+					(size 1.27 1.27)
+				)
+				(hide yes)
+			)
+		)
+		(property "Datasheet" ""
+			(at 58.42 55.88 0)
+			(effects
+				(font
+					(size 1.27 1.27)
+				)
+				(hide yes)
+			)
+		)
+		(property "Description" "Power symbol creates a global label with name \"GND\" , ground"
+			(at 58.42 55.88 0)
+			(effects
+				(font
+					(size 1.27 1.27)
+				)
+				(hide yes)
+			)
+		)
+		(pin "1"
+		)
+		(instances
+			(project "keyboard_v2"
+				(path "/e2360b7f-be71-48d9-b398-9f8cd45479d6/b599252a-0e44-4760-9c79-385d4380db60"
+					(reference "#PWR0305")
+					(unit 1)
+				)
+			)
+		)
+	)
+	(symbol
+		(lib_id "ANT3216A063R2400A:ANT3216A063R2400A")
+		(at 55.88 48.26 0)
 		(mirror y)
 		(unit 1)
@@
 		(on_board yes)
 		(dnp no)
-		(property "Reference" "AE302"
-			(at 62.23 38.7349 0)
-			(effects
-				(font
-					(size 1.27 1.27)
-				)
-				(justify left)
-			)
-		)
-		(property "Value" "Antenna_Shield"
-			(at 62.23 41.2749 0)
-			(effects
-				(font
-					(size 1.27 1.27)
-				)
-				(justify left)
-			)
-		)
-		(property "Footprint" "RF_Antenna:Texas_SWRA117D_2.4GHz_Right"
-			(at 66.04 38.1 0)
-			(effects
-				(font
-					(size 1.27 1.27)
-				)
-				(hide yes)
-			)
-		)
-		(property "Datasheet" "~"
-			(at 66.04 38.1 0)
-			(effects
-				(font
-					(size 1.27 1.27)
-				)
-				(hide yes)
-			)
-		)
-		(property "Description" "Antenna with extra pin for shielding"
-			(at 66.04 40.64 0)
-			(effects
-				(font
-					(size 1.27 1.27)
-				)
+		(fields_autoplaced yes)
+		(property "Reference" "ANT301"
+			(at 44.45 40.64 0)
+			(effects
+				(font
+					(size 1.27 1.27)
+				)
+			)
+		)
+		(property "Value" "ANT3216A063R2400A"
+			(at 44.45 43.18 0)
+			(effects
+				(font
+					(size 1.27 1.27)
+				)
+			)
+		)
+		(property "Footprint" "keyboard_footprints:ANTC3016X65N"
+			(at 36.83 143.18 0)
+			(effects
+				(font
+					(size 1.27 1.27)
+				)
+				(justify left top)
+				(hide yes)
+			)
+		)
+		(property "Datasheet" "https://media.digikey.com/pdf/Data%20Sheets/Yageo%20PDFs/ANT3216A063R2400A_Rev2014.pdf"
+			(at 36.83 243.18 0)
+			(effects
+				(font
+					(size 1.27 1.27)
+				)
+				(justify left top)
+				(hide yes)
+			)
+		)
+		(property "Description" "Antennas 1W, 2.45GHz, 3216"
+			(at 55.88 63.5 0)
+			(effects
+				(font
+					(size 1.27 1.27)
+				)
+				(hide yes)
+			)
+		)
+		(property "Height" "0.65"
+			(at 36.83 443.18 0)
+			(effects
+				(font
+					(size 1.27 1.27)
+				)
+				(justify left top)
+				(hide yes)
+			)
+		)
+		(property "Mouser Part Number" "603-ANT3216A063R2400"
+			(at 36.83 543.18 0)
+			(effects
+				(font
+					(size 1.27 1.27)
+				)
+				(justify left top)
+				(hide yes)
+			)
+		)
+		(property "Mouser Price/Stock" "https://www.mouser.co.uk/ProductDetail/Pulse-Electronics/ANT3216A063R2400A?qs=CqAAFKzD4h%252BYK9SO0hbvNw%3D%3D"
+			(at 36.83 643.18 0)
+			(effects
+				(font
+					(size 1.27 1.27)
+				)
+				(justify left top)
+				(hide yes)
+			)
+		)
+		(property "Manufacturer_Name" "Pulse Electronics"
+			(at 36.83 743.18 0)
+			(effects
+				(font
+					(size 1.27 1.27)
+				)
+				(justify left top)
+				(hide yes)
+			)
+		)
+		(property "Manufacturer_Part_Number" "ANT3216A063R2400A"
+			(at 36.83 843.18 0)
+			(effects
+				(font
+					(size 1.27 1.27)
+				)
+				(justify left top)
 				(hide yes)
 			)
@@
 		)
 		(pin "2"
+		)
+		(pin "3"
 		)
 		(instances
 			(project "keyboard_v2"
 				(path "/e2360b7f-be71-48d9-b398-9f8cd45479d6/b599252a-0e44-4760-9c79-385d4380db60"
-					(reference "AE302")
+					(reference "ANT301")
 					(unit 1)
 				)
@@
 		)
 	)
-	(symbol
-		(lib_id "power:GND")
-		(at 63.5 48.26 0)
-		(unit 1)
-		(exclude_from_sim no)
-		(in_bom yes)
-		(on_board yes)
-		(dnp no)
-		(fields_autoplaced yes)
-		(property "Reference" "#PWR0305"
-			(at 63.5 54.61 0)
-			(effects
-				(font
-					(size 1.27 1.27)
-				)
-				(hide yes)
-			)
-		)
-		(property "Value" "GND"
-			(at 63.5 53.34 0)
-			(effects
-				(font
-					(size 1.27 1.27)
-				)
-			)
-		)
-		(property "Footprint" ""
-			(at 63.5 48.26 0)
-			(effects
-				(font
-					(size 1.27 1.27)
-				)
-				(hide yes)
-			)
-		)
-		(property "Datasheet" ""
-			(at 63.5 48.26 0)
-			(effects
-				(font
-					(size 1.27 1.27)
-				)
-				(hide yes)
-			)
-		)
-		(property "Description" "Power symbol creates a global label with name \"GND\" , ground"
-			(at 63.5 48.26 0)
-			(effects
-				(font
-					(size 1.27 1.27)
-				)
-				(hide yes)
-			)
-		)
-		(pin "1"
-		)
-		(instances
-			(project "keyboard_v2"
-				(path "/e2360b7f-be71-48d9-b398-9f8cd45479d6/b599252a-0e44-4760-9c79-385d4380db60"
-					(reference "#PWR0305")
-					(unit 1)
-				)
-			)
-		)
-	)
 	(sheet
 		(at 68.58 71.12)
@@
 			)
 		)
-		(property "Sheetfile" "usb.kicad_sch"
+		(property "Sheetfile" "usb_right.kicad_sch"
 			(at 68.58 97.1046 0)
 			(effects
@@
 			(color 0 0 0 0.0000)
 		)
-		(property "Sheetname" "Keys Right"
+		(property "Sheetname" "Keys"
 			(at 195.58 39.9284 0)
 			(effects
@@
 			)
 		)
-		(pin "ANT" output
+		(pin "ANT" bidirectional
 			(at 68.58 48.26 180)
 			(effects
@@
 			(color 0 0 0 0.0000)
 		)
-		(property "Sheetname" "Main MCU Right"
+		(property "Sheetname" "Main MCU"
 			(at 144.78 39.9284 0)
 			(effects
