File: PCBs/keyboard_v2/bluetooth.kicad_sch (KiCad schematic)
At the start: 2 parts, among them U901 nRF52840-QFAA-F-R7

Commit message: V2 progress
Parts:
- added C903, C904: 12p, Capacitor_SMD:C_0402_1005Metric, symbol Device:C_Small
- added C905: 1p, Capacitor_SMD:C_0402_1005Metric, symbol Device:C_Small
- added C906: 1p2, Capacitor_SMD:C_0402_1005Metric, symbol Device:C_Small
- added C907, C908, C909, C910, C911: 100n, Capacitor_SMD:C_0402_1005Metric, symbol Device:C_Small
- added C912, C915: 1u, Capacitor_SMD:C_0402_1005Metric, symbol Device:C_Small
- added C913: 100p, Capacitor_SMD:C_0402_1005Metric, symbol Device:C_Small
- added C914: 47n, Capacitor_SMD:C_0402_1005Metric, symbol Device:C_Small
- added L901: 10u, Inductor_SMD:L_0402_1005Metric, symbol Device:L_Small
- added L902: 4n7, Inductor_SMD:L_0402_1005Metric, symbol Device:L_Small
- added L905: 2n2, Inductor_SMD:L_0402_1005Metric, symbol Device:L_Small
- added L906: 15n, Inductor_SMD:L_0402_1005Metric, symbol Device:L_Small
- added Y902: 32MHz, Crystal:Crystal_SMD_2016-4Pin_2.0x1.6mm, symbol Device:Crystal_GND24_Small
- renumbered AE901 to AE1001, U901 to U1001
Connections:
- net DEC1: now reaches U1001.1 (DEC1)
- net DEC1: now also C911.1
- net at U1001.12 (VDD_1): now also U1001.17 (VDD_2), U1001.25 (VDD_3), U1001.37 (VDD_4), U1001.48 (VDD_5), C907.1, C908.1, C909.1, C910.1, C912.1
- net RST: now reaches U1001.16 (P0.18/NRESET)
- net SWDIO: now reaches U1001.26 (SWDIO)
- net SWCLK: now reaches U1001.27 (SWDCLK)
- net RF1: now reaches U1001.31 (ANT)
- net RF1: now also L902.1
- net GND: now reaches U1001.32 (VSS_PA)
- net GND: now also U1001.45 (VSS_1), U1001.49 (VSS_2), C903.1, C904.1, C905.2, C906.2, C907.2, C908.2, C909.2, C910.2, C911.2, C912.2, C913.2, C914.2, C915.2, Y902.2, Y902.4
- net DEC4_6: now reaches U1001.33 (DEC6)
- net DEC4_6: now also U1001.46 (DEC4), C914.1, C915.1, L906.2
- net DEC3: now reaches U1001.34 (DEC3)
- net DEC3: now also C913.1
- net XC1: now reaches U1001.35 (XC1)
- net XC1: now also C903.2, Y902.3
- net XC2: now reaches U1001.36 (XC2)
- net XC2: now also C904.2, Y902.1
- net DCC1: now reaches U1001.47 (DCC)
- net DCC1: now also L901.1
- net ANT: now reaches AE1001.1 (A)
- net ANT: now also C906.1, L905.2
- new net DCC2: L901.2, L906.1
- new net RF2: C905.1, L902.2, L905.1
- no-connect marks 0 -> 28
Other:
- moved on the sheet: AE1001, U1001

Commit message: Display schematic done
Connections:
- net +1V8: now reaches C907.1, C908.1, C909.1, C910.1, C912.1, U1001.12 (VDD_1), U1001.17 (VDD_2), U1001.25 (VDD_3), U1001.37 (VDD_4), U1001.48 (VDD_5)
Changed lines of the file:
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@@
 		(color 0 0 0 0)
 	)
+	(junction
+		(at 198.12 127)
+		(diameter 0)
+		(color 0 0 0 0)
+	)
 	(no_connect
 		(at 104.14 91.44)
@@
 		(pts
 			(xy 157.48 111.76) (xy 157.48 114.3)
+		)
+		(stroke
+			(width 0)
+			(type default)
+		)
+	)
+	(wire
+		(pts
+			(xy 198.12 124.46) (xy 198.12 127)
 		)
 		(stroke
@@
 					(unit 1)
 				)
+			)
+		)
+	)
+	(symbol
+		(lib_id "power:+1V8")
+		(at 198.12 124.46 0)
+		(mirror y)
+		(unit 1)
+		(exclude_from_sim no)
+		(in_bom yes)
+		(on_board yes)
+		(dnp no)
+		(fields_autoplaced yes)
+		(property "Reference" "#PWR0908"
+			(at 198.12 128.27 0)
+			(effects
+				(font
+					(size 1.27 1.27)
+				)
+				(hide yes)
+			)
+		)
+		(property "Value" "+1V8"
+			(at 198.12 119.38 0)
+			(effects
+				(font
+					(size 1.27 1.27)
+				)
+			)
+		)
+		(property "Footprint" ""
+			(at 198.12 124.46 0)
+			(effects
+				(font
+					(size 1.27 1.27)
+				)
+				(hide yes)
+			)
+		)
+		(property "Datasheet" ""
+			(at 198.12 124.46 0)
+			(effects
+				(font
+					(size 1.27 1.27)
+				)
+				(hide yes)
+			)
+		)
+		(property "Description" "Power symbol creates a global label with name \"+1V8\""
+			(at 198.12 124.46 0)
+			(effects
+				(font
+					(size 1.27 1.27)
+				)
+				(hide yes)
+			)
+		)
+		(pin "1"
+		)
+		(instances
+			(project "keyboard_v2"
+				(path "/e2360b7f-be71-48d9-b398-9f8cd45479d6/b599252a-0e44-4760-9c79-385d4380db60/bf97ba9d-665b-4380-a56f-118a3ac4ddf1"
+					(reference "#PWR0908")
+					(unit 1)
+				)
+				(path "/e2360b7f-be71-48d9-b398-9f8cd45479d6/8d5749a2-4d36-4f17-8c57-9c8b87d773d6/d174db9b-07f6-4c79-87e9-921db730cdfb"
+					(reference "#PWR01008")
+					(unit 1)
+				)

Commit message: V2 Schematic mostly done
Parts:
- removed AE1001: Antenna, RF_Antenna:Texas_SWRA117D_2.4GHz_Left, symbol Device:Antenna
- renumbered C903 to C1003, C904 to C1004, C905 to C1005, C906 to C1006, C907 to C1007, C908 to C1008, C909 to C1009, C910 to C1010, C911 to C1011, C912 to C1012, C913 to C1013, C914 to C1014, C915 to C1015, L901 to L1001, L902 to L1002, L905 to L1005, L906 to L1006, Y902 to Y1002
Connections:
- no-connect marks 28 -> 27

Commit message: Layout in progress
Changed lines of the file:
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@@
 	(wire
 		(pts
-			(xy 200.66 53.34) (xy 208.28 53.34)
+			(xy 200.66 53.34) (xy 210.82 53.34)
 		)
 		(stroke
@@
 			)
 			(justify left bottom)
-		)
-	)
-	(hierarchical_label "ANT"
-		(shape output)
-		(at 208.28 53.34 0)
-		(fields_autoplaced yes)
-		(effects
-			(font
-				(size 1.27 1.27)
-			)
-			(justify left)
 		)
 	)
@@
 		)
 	)
+	(hierarchical_label "ANT"
+		(shape bidirectional)
+		(at 210.82 53.34 0)
+		(fields_autoplaced yes)
+		(effects
+			(font
+				(size 1.27 1.27)
+			)
+			(justify left)
+		)
+	)

Commit message: 279 Unrouted
Connections:
- net UART_RX: now also U1001.23 (P0.24)
- net UART_TX: now also U1001.22 (P0.23)
Changed lines of the file:
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@@
+	)
+	(no_connect
+		(at 104.14 132.08)
 	)
 	(no_connect
@@
 	)
 	(no_connect
-		(at 104.14 132.08)
-	)
-	(no_connect
 		(at 104.14 86.36)
 	)
@@
 	)
 	(no_connect
-		(at 104.14 111.76)
-	)
-	(no_connect
-		(at 104.14 114.3)
-	)
-	(no_connect
 		(at 104.14 134.62)
 	)
 	(no_connect
+		(at 104.14 63.5)
+	)
+	(no_connect
 		(at 104.14 71.12)
 	)
@@
 	)
 	(no_connect
+		(at 104.14 68.58)
+	)
+	(no_connect
 		(at 104.14 129.54)
 	)
 	(no_connect
-		(at 104.14 68.58)
-	)
-	(no_connect
 		(at 104.14 83.82)
 	)
@@
 	)
 	(no_connect
+		(at 104.14 60.96)
+	)
+	(no_connect
 		(at 104.14 106.68)
 	)
@@
 	(wire
 		(pts
+			(xy 101.6 114.3) (xy 104.14 114.3)
+		)
+		(stroke
+			(width 0)
+			(type default)
+		)
+	)
+	(wire
+		(pts
 			(xy 175.26 71.12) (xy 175.26 73.66)
 		)
@@
 		(pts
 			(xy 177.8 101.6) (xy 177.8 99.06)
+		)
+		(stroke
+			(width 0)
+			(type default)
+		)
+	)
+	(wire
+		(pts
+			(xy 101.6 111.76) (xy 104.14 111.76)
 		)
 		(stroke
@@
 		)
 	)
-	(hierarchical_label "UART_RX"
-		(shape input)
-		(at 55.88 91.44 180)
+	(hierarchical_label "UART_TX"
+		(shape output)
+		(at 101.6 111.76 180)
 		(fields_autoplaced yes)
 		(effects
@@
 		)
 	)
+	(hierarchical_label "UART_RX"
+		(shape input)
+		(at 101.6 114.3 180)
+		(fields_autoplaced yes)
+		(effects
+			(font
+				(size 1.27 1.27)
+			)
+			(justify right)
+		)
+	)
 	(hierarchical_label "ANT"
 		(shape bidirectional)
@@
 		)
 	)
-	(hierarchical_label "UART_TX"
-		(shape output)
-		(at 55.88 88.9 180)
-		(fields_autoplaced yes)
-		(effects
-			(font
-				(size 1.27 1.27)
-			)
-			(justify right)
-		)
-	)
