File: PCBs/keyboard_v2/main_mcu_left.kicad_sch (KiCad schematic)
At the start: 28 parts, among them U1301 STM32U5G9ZJJ6Q, U1302 M24256X-FCU6T_VF, Y1301 16MHz

Commit message: V2 progress
Parts:
- removed C1301, C1302: 6p, Capacitor_SMD:C_0402_1005Metric, symbol Device:C_Small
- removed Y1301: 16MHz, Crystal:Crystal_SMD_2016-4Pin_2.0x1.6mm, symbol Device:Crystal_GND24_Small
- added C1323, C1324: 12p, Capacitor_SMD:C_0402_1005Metric, symbol Device:C_Small
- added Y1302: 32MHz, Crystal:Crystal_SMD_2016-4Pin_2.0x1.6mm, symbol Device:Crystal_GND24_Small
Connections:
- net GND: now also C1323.1, C1324.1, Y1302.2, Y1302.4
- net OSC_IN: now also C1323.2, Y1302.3
- net OSC_OUT: now also C1324.2, Y1302.1

Commit message: V2 Schematic mostly done
Parts:
- U1302: footprint watch_footprints:BGA4C50P2X2_70X98X33 -> keyboard_footprints:BGA4C50P2X2_70X98X33
Connections:
- net +1V8: now also R1301.1, R1302.1, U1302.A1 (VCC); no longer C1313.1, C1315.1, U1301.E6 (VDDIO2)
- net +3V3: now also C1313.1, C1315.1, U1301.E6 (VDDIO2); no longer R1301.1, R1302.1, U1302.A1 (VCC)
- net DSI_CKN: now also U1301.F1 (DSI_CKN)
- net DSI_CKP: now also U1301.F2 (DSI_CKP)
- net DSI_D0N: now also U1301.E1 (DSI_D0N)
- net DSI_D0P: now also U1301.E2 (DSI_D0P)
- net OSC_IN: now also U1301.H2 (PH0-OSC_IN)
- net OSC_OUT: now also U1301.J1 (PH1-OSC_OUT)
- net RST: now also U1301.J2 (NRST)
- no-connect marks 0 -> 2
Other:
- note added: "ENCODER PINS MUST BE 5V TOLERANT"
- moved on the sheet: U1301B

Commit message: Schematic mostly done, moving onto PCB
Parts:
- removed C1318, C1320: 100n, Capacitor_SMD:C_0201_0603Metric, symbol Device:C_Small
- added C1301, C1302: 100n, Capacitor_SMD:C_0402_1005Metric, symbol Device:C_Small
- C1303, C1304, C1305, C1306, C1309, C1310, C1311, C1312, C1313, C1314, C1316, C1317, C1321, C1322: footprint Capacitor_SMD:C_0201_0603Metric -> Capacitor_SMD:C_0402_1005Metric
Connections:
- net +1V8: now also C1301.1, C1302.1; no longer C1311.1
- net +3V3: now also C1311.1
- net DSI_TE: now also U1301.C5 (PB7)
- net GND: now also C1301.2, C1302.2
- net SWCLK: now also U1301.B11 (PA14)
- net SWDIO: now also U1301.C10 (PA13)
- net USB_DN: now also U1301.C12 (PA11)
- net USB_DP: now also U1301.C11 (PA12)
- no-connect marks 2 -> 4

Commit message: Placement done
Parts:
- C1307: footprint Capacitor_SMD:C_0201_0603Metric -> Capacitor_SMD:C_0402_1005Metric
Changed lines of the file:
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@@
 			)
 		)
-		(property "Footprint" "Capacitor_SMD:C_0201_0603Metric"
+		(property "Footprint" "Capacitor_SMD:C_0402_1005Metric"
 			(at 76.2 264.16 0)
 			(effects

Commit message: 279 Unrouted
Connections:
- net SCL is gone; now on net PWR_SCL: R1302.2, U1302.A2 (SCL)
- net SDA is gone; now on net PWR_SDA: R1301.2, U1302.B1 (SDA)
Changed lines of the file:
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@@
+	(wire
+		(pts
+			(xy 325.12 144.78) (xy 337.82 144.78)
+		)
+		(stroke
+			(width 0)
+			(type default)
+		)
+	)
 	(wire
 		(pts
@@
 		(pts
 			(xy 58.42 236.22) (xy 58.42 233.68)
+		)
+		(stroke
+			(width 0)
+			(type default)
+		)
+	)
+	(wire
+		(pts
+			(xy 325.12 147.32) (xy 337.82 147.32)
 		)
 		(stroke
@@
 		)
 	)
+	(label "SCL"
+		(at 330.2 144.78 0)
+		(fields_autoplaced yes)
+		(effects
+			(font
+				(size 1.27 1.27)
+			)
+			(justify left bottom)
+		)
+	)
 	(label "OSC_IN"
 		(at 210.82 53.34 180)
@@
 		)
 	)
+	(label "SDA"
+		(at 330.2 147.32 0)
+		(fields_autoplaced yes)
+		(effects
+			(font
+				(size 1.27 1.27)
+			)
+			(justify left bottom)
+		)
+	)
 	(label "VREF+"
 		(at 276.86 205.74 180)
@@
 	(hierarchical_label "PWR_SDA"
 		(shape bidirectional)
-		(at 345.44 86.36 0)
-		(fields_autoplaced yes)
-		(effects
-			(font
-				(size 1.27 1.27)
-			)
-			(justify left)
+		(at 325.12 147.32 180)
+		(fields_autoplaced yes)
+		(effects
+			(font
+				(size 1.27 1.27)
+			)
+			(justify right)
 		)
 	)
@@
 		)
 	)
+	(hierarchical_label "SCL_TP"
+		(shape output)
+		(at 353.06 149.86 180)
+		(fields_autoplaced yes)
+		(effects
+			(font
+				(size 1.27 1.27)
+			)
+			(justify right)
+		)
+	)
 	(hierarchical_label "KEY_A6"
 		(shape input)
@@
 	(hierarchical_label "PWR_SCL"
 		(shape output)
-		(at 345.44 83.82 0)
-		(fields_autoplaced yes)
-		(effects
-			(font
-				(size 1.27 1.27)
-			)
-			(justify left)
+		(at 325.12 144.78 180)
+		(fields_autoplaced yes)
+		(effects
+			(font
+				(size 1.27 1.27)
+			)
+			(justify right)
 		)
 	)
@@
 	(hierarchical_label "SDA_TP"
 		(shape bidirectional)
-		(at 345.44 147.32 0)
-		(fields_autoplaced yes)
-		(effects
-			(font
-				(size 1.27 1.27)
-			)
-			(justify left)
+		(at 353.06 152.4 180)
+		(fields_autoplaced yes)
+		(effects
+			(font
+				(size 1.27 1.27)
+			)
+			(justify right)
 		)
 	)
@@
 		(fields_autoplaced yes)
 		(effects
-			(font
-				(size 1.27 1.27)
-			)
-			(justify left)
-		)
-	)
-	(hierarchical_label "SCL_TP"
-		(shape output)
-		(at 345.44 144.78 0)
-		(fields_autoplaced yes)
-		(effects
