File: PCBs/keyboard_v2/main_mcu_right.kicad_sch (KiCad schematic)
At the start: 28 parts, among them U801 STM32U5G9ZJJ6Q, U802 M24256X-FCU6T_VF, Y802 32MHz

Commit message: 249 Unrouted
Connections:
- net BLE_RST: now also U801.M4 (PB1)
- net USB_RST: now also U801.M3 (PA6)
- net USB_UART_RX: now also U801.A8 (PG10)
- net USB_UART_TX: now also U801.B7 (PG9)
Changed lines of the file:
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@@
+	(wire
+		(pts
+			(xy 27.94 68.58) (xy 43.18 68.58)
+		)
+		(stroke
+			(width 0)
+			(type default)
+		)
+	)
 	(wire
 		(pts
@@
 	(wire
 		(pts
+			(xy 27.94 101.6) (xy 43.18 101.6)
+		)
+		(stroke
+			(width 0)
+			(type default)
+		)
+	)
+	(wire
+		(pts
 			(xy 363.22 195.58) (xy 363.22 203.2)
 		)
@@
 	(wire
 		(pts
+			(xy 139.7 119.38) (xy 149.86 119.38)
+		)
+		(stroke
+			(width 0)
+			(type default)
+		)
+	)
+	(wire
+		(pts
 			(xy 256.54 228.6) (xy 254 228.6)
 		)
@@
 		(pts
 			(xy 256.54 208.28) (xy 256.54 210.82)
+		)
+		(stroke
+			(width 0)
+			(type default)
+		)
+	)
+	(wire
+		(pts
+			(xy 139.7 116.84) (xy 149.86 116.84)
 		)
 		(stroke
@@
 		)
 	)
-	(hierarchical_label "USB_UART_RX"
-		(shape input)
-		(at 312.42 81.28 0)
-		(fields_autoplaced yes)
-		(effects
-			(font
-				(size 1.27 1.27)
-			)
-			(justify left)
-		)
-	)
 	(hierarchical_label "NEOPIXEL"
 		(shape output)
@@
 		)
 	)
+	(hierarchical_label "USB_UART_RX"
+		(shape input)
+		(at 139.7 119.38 180)
+		(fields_autoplaced yes)
+		(effects
+			(font
+				(size 1.27 1.27)
+			)
+			(justify right)
+		)
+	)
 	(hierarchical_label "KEY_E6"
 		(shape input)
@@
 	(hierarchical_label "USB_RST"
 		(shape output)
-		(at 312.42 86.36 0)
-		(fields_autoplaced yes)
-		(effects
-			(font
-				(size 1.27 1.27)
-			)
-			(justify left)
+		(at 27.94 68.58 180)
+		(fields_autoplaced yes)
+		(effects
+			(font
+				(size 1.27 1.27)
+			)
+			(justify right)
 		)
 	)
@@
 	(hierarchical_label "USB_UART_TX"
 		(shape output)
-		(at 312.42 83.82 0)
-		(fields_autoplaced yes)
-		(effects
-			(font
-				(size 1.27 1.27)
-			)
-			(justify left)
+		(at 139.7 116.84 180)
+		(fields_autoplaced yes)
+		(effects
+			(font
+				(size 1.27 1.27)
+			)
+			(justify right)
 		)
 	)
@@
 	(hierarchical_label "BLE_RST"
 		(shape output)
-		(at 312.42 71.12 0)
-		(fields_autoplaced yes)
-		(effects
-			(font
-				(size 1.27 1.27)
-			)
-			(justify left)
-		)
-	)
+		(at 27.94 101.6 180)
+		(fields_autoplaced yes)
+		(effects
+			(font
+				(size 1.27 1.27)
+			)
+			(justify right)
+		)
+	)
