File: PCBs/keyboard_v2/usb_right.kicad_sch (KiCad schematic)
At the start: 22 parts, among them J601 USB4510-03-1-A, J602 USB4510-03-1-A, J603 GSB12J21C1EU, U601 USBLC6-4SC6, U602 USBLC6-4SC6, U603 USBLC6-4SC6, U604 STM32G0B1KBUx, U605 USB2533-1080AEN, Y601 CX2016SA24000D0HLLG3

Commit message: Layout progress
Parts:
- added U606: USBLC6-4SC6, Package_TO_SOT_SMD:SOT-23-6, symbol Power_Protection:USBLC6-4SC6
Connections:
- net GND: now also U606.2 (GND)
- net USB0_RX: now also U606.6 (I/O4)
- net USB0_TX: now also U606.4 (I/O3)
- net USB1_RX: now also U606.3 (I/O2)
- net USB1_TX: now also U606.1 (I/O1)
- net VBUS: now also U606.5 (VBUS)

Commit message: 339 Unrouted
Connections:
- net +3V3: no longer U605.26 (RESET_N)
- net USB2_DN: now also U603.3 (I/O2); no longer U603.1 (I/O1)
- net USB2_DP: now also U603.1 (I/O1); no longer U603.3 (I/O2)
- new net USB_RST: U605.26 (RESET_N)
Changed lines of the file:
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@@
 	(wire
 		(pts
-			(xy 203.2 58.42) (xy 208.28 58.42)
+			(xy 124.46 91.44) (xy 137.16 91.44)
 		)
 		(stroke
@@
 	(wire
 		(pts
-			(xy 132.08 91.44) (xy 137.16 91.44)
+			(xy 203.2 58.42) (xy 208.28 58.42)
 		)
 		(stroke
@@
 	(wire
 		(pts
+			(xy 5.08 88.9) (xy 17.78 88.9)
+		)
+		(stroke
+			(width 0)
+			(type default)
+		)
+	)
+	(wire
+		(pts
 			(xy 35.56 81.28) (xy 48.26 81.28)
 		)
@@
 	(wire
 		(pts
-			(xy 132.08 88.9) (xy 132.08 91.44)
-		)
-		(stroke
-			(width 0)
-			(type default)
-		)
-	)
-	(wire
-		(pts
 			(xy 231.14 132.08) (xy 231.14 134.62)
 		)
@@
 		)
 	)
+	(label "USB_RST"
+		(at 5.08 88.9 0)
+		(fields_autoplaced yes)
+		(effects
+			(font
+				(size 1.27 1.27)
+			)
+			(justify left bottom)
+		)
+	)
 	(label "USB2_DN"
 		(at 124.46 58.42 0)
@@
 	)
 	(label "USB2_DN"
-		(at 243.84 139.7 0)
+		(at 243.84 142.24 0)
 		(fields_autoplaced yes)
 		(effects
@@
 		)
 	)
+	(label "USB_RST"
+		(at 124.46 91.44 0)
+		(fields_autoplaced yes)
+		(effects
+			(font
+				(size 1.27 1.27)
+			)
+			(justify left bottom)
+		)
+	)
 	(label "SDA"
 		(at 124.46 73.66 0)
@@
 	)
 	(label "USB2_DP"
-		(at 243.84 142.24 0)
+		(at 243.84 139.7 0)
 		(fields_autoplaced yes)
 		(effects
@@
 					(unit 1)
 				)
-			)
-		)
-	)
-	(symbol
-		(lib_id "power:+3V3")
-		(at 132.08 88.9 0)
-		(unit 1)
-		(exclude_from_sim no)
-		(in_bom yes)
-		(on_board yes)
-		(dnp no)
-		(fields_autoplaced yes)
-		(property "Reference" "#PWR0622"
-			(at 132.08 92.71 0)
-			(effects
-				(font
-					(size 1.27 1.27)
-				)
-				(hide yes)
-			)
-		)
-		(property "Value" "+3V3"
-			(at 132.08 83.82 0)
-			(effects
-				(font
-					(size 1.27 1.27)
-				)
-			)
-		)
-		(property "Footprint" ""
-			(at 132.08 88.9 0)
-			(effects
-				(font
-					(size 1.27 1.27)
-				)
-				(hide yes)
-			)
-		)
-		(property "Datasheet" ""
-			(at 132.08 88.9 0)
-			(effects
-				(font
-					(size 1.27 1.27)
-				)
-				(hide yes)
-			)
-		)
-		(property "Description" "Power symbol creates a global label with name \"+3V3\""
-			(at 132.08 88.9 0)
-			(effects
-				(font
-					(size 1.27 1.27)
-				)
-				(hide yes)
-			)
-		)
-		(pin "1"
-		)
-		(instances
-			(project "keyboard_v2"
-				(path "/e2360b7f-be71-48d9-b398-9f8cd45479d6/b599252a-0e44-4760-9c79-385d4380db60/2fa754a4-db8f-4839-bd38-632dd798fa1f"
-					(reference "#PWR0622")
-					(unit 1)
-				)

Commit message: 249 Unrouted
Connections:
- net +3V3: now also U604.20 (PC6)
- net UART_RX: now also U604.8 (PA1)
- net UART_TX: now also U604.7 (PA0)
Changed lines of the file:
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@@
 	(wire
 		(pts
+			(xy 99.06 55.88) (xy 83.82 55.88)
+		)
+		(stroke
+			(width 0)
+			(type default)
+		)
+	)
+	(wire
+		(pts
 			(xy 205.74 45.72) (xy 203.2 45.72)
 		)
@@
 	(wire
 		(pts
+			(xy 99.06 58.42) (xy 83.82 58.42)
+		)
+		(stroke
+			(width 0)
+			(type default)
+		)
+	)
+	(wire
+		(pts
 			(xy 142.24 144.78) (xy 142.24 147.32)
 		)
@@
 	(wire
 		(pts
+			(xy 45.72 60.96) (xy 48.26 60.96)
+		)
+		(stroke
+			(width 0)
+			(type default)
+		)
+	)
+	(wire
+		(pts
 			(xy 205.74 43.18) (xy 205.74 45.72)
 		)
@@
 	(wire
 		(pts
+			(xy 45.72 48.26) (xy 45.72 60.96)
+		)
+		(stroke
+			(width 0)
+			(type default)
+		)
+	)
+	(wire
+		(pts
 			(xy 109.22 154.94) (xy 96.52 154.94)
 		)
@@
 	(hierarchical_label "UART_TX"
 		(shape output)
-		(at 35.56 104.14 180)
+		(at 99.06 55.88 0)
 		(fields_autoplaced yes)
 		(effects
@@
 				(size 1.27 1.27)
 			)
-			(justify right)
+			(justify left)
 		)
 	)
@@
 	(hierarchical_label "UART_RX"
 		(shape input)
-		(at 35.56 106.68 180)
+		(at 99.06 58.42 0)
 		(fields_autoplaced yes)
 		(effects
@@
 				(size 1.27 1.27)
 			)
-			(justify right)
+			(justify left)
 		)
 	)
@@
 					(unit 1)
 				)
+			)
+		)
+	)
+	(symbol
+		(lib_id "power:+3V3")
+		(at 45.72 48.26 0)
+		(unit 1)
+		(exclude_from_sim no)
+		(in_bom yes)
+		(on_board yes)
+		(dnp no)
+		(fields_autoplaced yes)
+		(property "Reference" "#PWR0622"
+			(at 45.72 52.07 0)
+			(effects
+				(font
+					(size 1.27 1.27)
+				)
+				(hide yes)
+			)
+		)
+		(property "Value" "+3V3"
+			(at 45.72 43.18 0)
+			(effects
+				(font
+					(size 1.27 1.27)
+				)
+			)
+		)
+		(property "Footprint" ""
+			(at 45.72 48.26 0)
+			(effects
+				(font
+					(size 1.27 1.27)
+				)
+				(hide yes)
+			)
+		)
+		(property "Datasheet" ""
+			(at 45.72 48.26 0)
+			(effects
+				(font
+					(size 1.27 1.27)
+				)
+				(hide yes)
+			)
+		)
+		(property "Description" "Power symbol creates a global label with name \"+3V3\""
+			(at 45.72 48.26 0)
+			(effects
+				(font
+					(size 1.27 1.27)
+				)
+				(hide yes)
+			)
+		)
+		(pin "1"
+		)
+		(instances
+			(project "keyboard_v2"
+				(path "/e2360b7f-be71-48d9-b398-9f8cd45479d6/b599252a-0e44-4760-9c79-385d4380db60/2fa754a4-db8f-4839-bd38-632dd798fa1f"
+					(reference "#PWR0622")
+					(unit 1)
+				)
