File: PCBs/keyboard-v3/right-control-board/debug-connector.kicad_sch (KiCad schematic)
At the start: 1 part, among them J501 Conn_02x08_Odd_Even

Commit message: Right control board placement and schematic done
Connections:
- net CTRL.SWCLK: now also J501.2 (Pin_2); no longer J501.1 (Pin_1)
- net CTRL.SWDIO: now also J501.1 (Pin_1); no longer J501.2 (Pin_2)
- net KEYS.SWCLK: now also J501.10 (Pin_10); no longer J501.9 (Pin_9)
- net KEYS.SWDIO: now also J501.9 (Pin_9); no longer J501.10 (Pin_10)
- net KNOB.SWCLK: now also J501.6 (Pin_6); no longer J501.5 (Pin_5)
- net KNOB.SWDIO: now also J501.5 (Pin_5); no longer J501.6 (Pin_6)
Changed lines of the file:
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@@
 	)
 	(label "CTRL.SWDIO"
-		(at 175.26 91.44 180)
+		(at 127 91.44 0)
+		(effects
+			(font
+				(size 1.27 1.27)
+			)
+			(justify left bottom)
+		)
+	)
+	(label "KEYS.SWCLK"
+		(at 175.26 101.6 180)
 		(effects
 			(font
@@
 			)
 			(justify right bottom)
-		)
-	)
-	(label "KEYS.SWCLK"
-		(at 127 101.6 0)
-		(effects
-			(font
-				(size 1.27 1.27)
-			)
-			(justify left bottom)
 		)
 	)
@@
 	)
 	(label "CTRL.SWCLK"
-		(at 127 91.44 0)
+		(at 175.26 91.44 180)
+		(effects
+			(font
+				(size 1.27 1.27)
+			)
+			(justify right bottom)
+		)
+	)
+	(label "KNOB.SWDIO"
+		(at 127 96.52 0)
 		(effects
 			(font
@@
 			)
 			(justify left bottom)
-		)
-	)
-	(label "KNOB.SWDIO"
-		(at 175.26 96.52 180)
-		(effects
-			(font
-				(size 1.27 1.27)
-			)
-			(justify right bottom)
 		)
 	)
@@
 	)
 	(label "KNOB.SWCLK"
-		(at 127 96.52 0)
+		(at 175.26 96.52 180)
+		(effects
+			(font
+				(size 1.27 1.27)
+			)
+			(justify right bottom)
+		)
+	)
+	(label "KEYS.SWDIO"
+		(at 127 101.6 0)
 		(effects
 			(font
@@
 		)
 	)
-	(label "KEYS.SWDIO"
-		(at 175.26 101.6 180)
-		(effects
-			(font
-				(size 1.27 1.27)
-			)
-			(justify right bottom)
-		)
-	)

Commit message: Right control board routing finished
Connections:
- net VBUS renamed +VSYS
Changed lines of the file:
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@@
 	)
 	(symbol
-		(lib_id "power:VBUS")
+		(lib_id "PWR-SYM:+VSYS")
 		(at 193.04 106.68 0)
 		(unit 1)
@@
 			)
 		)
-		(property "Value" "VBUS"
+		(property "Value" "+VSYS"
 			(at 193.04 101.6 0)
 			(effects
@@
 			)
 		)
-		(property "Description" "Power symbol creates a global label with name \"VBUS\""
+		(property "Description" "Power symbol creates a global label with name \"+VSYS\""
 			(at 193.04 106.68 0)
 			(effects
