File: PCBs/keyboard-v3/right-key-board/keys.kicad_sch (KiCad schematic)
At the start: 58 parts, among them Q201 DMN21D2UFB-7B, SW201 SW_DIP_x01, SW202 SW_DIP_x01, SW203 SW_DIP_x01, SW204 SW_DIP_x01, SW205 SW_DIP_x01, SW206 SW_DIP_x01, SW207 SW_DIP_x01, SW208 SW_DIP_x01, SW209 SW_DIP_x01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

Commit message: Right daughter boards finished
Connections:
- net VBUS renamed +5V

Commit message: Added mounting holes
Parts:
- renumbered D205 to D202, D209 to D203, D213 to D204, D217 to D205, D221 to D206, D202 to D207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
