File: PCBs/keyboard-v3/left-key-board/mcu.kicad_sch (KiCad schematic)
At the start: 11 parts, among them J301 F31Z1A7H111008, U301 STM32U031C6Ux

Commit message: Left control board done
Changed lines of the file:
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@@
 	(text_box "PB5:\nLOW = Left\nHIGH = Right\n\nPB6:\nLOW = Knob\nHIGH = Keys\n\n(Internal pullups)"
 		(exclude_from_sim no)
-		(at 55.88 104.14 0)
+		(at 53.34 104.14 0)
 		(size 20.32 20.32)
 		(margins 0.9525 0.9525 0.9525 0.9525)
@@
 	(text_box "An interrupt can be sent to the control board via PA15. The firmware must check no debugger is connected first."
 		(exclude_from_sim no)
-		(at 58.42 78.74 0)
+		(at 53.34 78.74 0)
 		(size 22.86 12.7)
 		(margins 0.9525 0.9525 0.9525 0.9525)
