File: PCBs/keyboard-v3/left-key-board/left-key-board.kicad_pcb (KiCad board)
At the start: 2 copper layers, 116 x 86 mm, 73 parts, among them J301 F31Z1A7H111008, Q201 DMN21D2UFB-7B, SW201 SW_DIP_x01, SW202 SW_DIP_x01, SW203 SW_DIP_x01, SW204 SW_DIP_x01, SW205 SW_DIP_x01, SW206 SW_DIP_x01, SW207 SW_DIP_x01, SW208 SW_DIP_x01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

Commit message: Left control board done
Parts:
- turned J301 to 0 degrees
Routing:
- net /MCU/SWDIO/~{INT}: track 24.0 -> 17.0 mm, vias 0 -> 2
- net /MCU/TX: track 16.5 -> 21.3 mm
- net /MCU/SWCLK: track 27.8 -> 31.8 mm
- net +3V3: track 39.7 -> 43.3 mm
- net GND: track 127.0 -> 129.8 mm, vias 89 -> 90
- net /MCU/~{RST}: track 35.6 -> 33.8 mm
- net /Keys/NEOPIXEL: track 17.5 -> 16.2 mm
- net /MCU/RX: track 16.9 -> 17.5 mm

Commit message: Keyboard v3 hardware done
Other:
- board text added: "Keyboard v3 Left Key Board Ben Smith 2026"
