File: PCBs/keyboard-v3/debug-breakout/debug-breakout.kicad_sch (KiCad schematic)
At the start: 4 parts, among them J101 Conn_ST_STDC14, J102 Conn_ST_STDC14, J103 Conn_ST_STDC14, J501 Conn_02x08_Odd_Even

Commit message: Right control board placement and schematic done
Connections:
- net CTRL.SWCLK: now also J501.2 (Pin_2); no longer J501.1 (Pin_1)
- net CTRL.SWDIO: now also J501.1 (Pin_1); no longer J501.2 (Pin_2)
- net KEYS.SWCLK: now also J501.10 (Pin_10); no longer J501.9 (Pin_9)
- net KEYS.SWDIO: now also J501.9 (Pin_9); no longer J501.10 (Pin_10)
- net KNOB.SWCLK: now also J501.6 (Pin_6); no longer J501.5 (Pin_5)
- net KNOB.SWDIO: now also J501.5 (Pin_5); no longer J501.6 (Pin_6)
Changed lines of the file:
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@@
 	)
 	(label "CTRL.SWDIO"
-		(at 226.06 93.98 180)
+		(at 177.8 93.98 0)
+		(effects
+			(font
+				(size 1.27 1.27)
+			)
+			(justify left bottom)
+		)
+	)
+	(label "KEYS.SWCLK"
+		(at 226.06 104.14 180)
 		(effects
 			(font
@@
 			)
 			(justify right bottom)
-		)
-	)
-	(label "KEYS.SWCLK"
-		(at 177.8 104.14 0)
-		(effects
-			(font
-				(size 1.27 1.27)
-			)
-			(justify left bottom)
 		)
 	)
@@
 	)
 	(label "CTRL.SWCLK"
-		(at 177.8 93.98 0)
+		(at 226.06 93.98 180)
+		(effects
+			(font
+				(size 1.27 1.27)
+			)
+			(justify right bottom)
+		)
+	)
+	(label "KEYS.SWDIO"
+		(at 177.8 104.14 0)
 		(effects
 			(font
@@
 		)
 	)
-	(label "KEYS.SWDIO"
-		(at 226.06 104.14 180)
+	(label "KNOB.SWCLK"
+		(at 226.06 99.06 180)
 		(effects
 			(font
@@
 			)
 			(justify right bottom)
-		)
-	)
-	(label "KNOB.SWCLK"
-		(at 177.8 99.06 0)
-		(effects
-			(font
-				(size 1.27 1.27)
-			)
-			(justify left bottom)
 		)
 	)
@@
 	)
 	(label "KNOB.SWDIO"
-		(at 226.06 99.06 180)
+		(at 177.8 99.06 0)
 		(effects
 			(font
 				(size 1.27 1.27)
 			)
-			(justify right bottom)
+			(justify left bottom)
 		)
 	)

Commit message: Finished debug breakout board and added 5V voltage sensing to key board
Connections:
- net +3V3: now also J501.1 (Pin_1); no longer J501.15 (Pin_15)
- net CTRL.SWCLK: now also J501.16 (Pin_16); no longer J501.2 (Pin_2)
- net CTRL.SWDIO: now also J501.15 (Pin_15); no longer J501.1 (Pin_1)
- net GND: now also J501.13 (Pin_13), J501.5 (Pin_5), J501.9 (Pin_9); no longer J501.11 (Pin_11), J501.3 (Pin_3), J501.7 (Pin_7)
- net KEYS.RX: now also J501.6 (Pin_6); no longer J501.12 (Pin_12)
- net KEYS.SWCLK: now also J501.8 (Pin_8); no longer J501.10 (Pin_10)
- net KEYS.SWDIO: now also J501.7 (Pin_7); no longer J501.9 (Pin_9)
- net KNOB.RX: now also J501.10 (Pin_10); no longer J501.8 (Pin_8)
- net KNOB.SWCLK: now also J501.12 (Pin_12); no longer J501.6 (Pin_6)
- net KNOB.SWDIO: now also J501.11 (Pin_11); no longer J501.5 (Pin_5)
- net VBUS: now also J501.2 (Pin_2); no longer J501.16 (Pin_16)
- net ~{RST}: now also J501.3 (Pin_3); no longer J501.13 (Pin_13)

Commit message: Keyboard v3 hardware done
Connections:
- net +3V3: now also J501.2 (Pin_2); no longer J501.1 (Pin_1)
- net CTRL.SWCLK: now also J501.15 (Pin_15); no longer J501.16 (Pin_16)
- net CTRL.SWDIO: now also J501.16 (Pin_16); no longer J501.15 (Pin_15)
- net GND: now also J501.10 (Pin_10), J501.3 (Pin_3), J501.6 (Pin_6); no longer J501.4 (Pin_4), J501.5 (Pin_5), J501.9 (Pin_9)
- net KEYS.RX: now also J501.5 (Pin_5); no longer J501.6 (Pin_6)
- net KEYS.SWCLK: now also J501.7 (Pin_7); no longer J501.8 (Pin_8)
- net KEYS.SWDIO: now also J501.8 (Pin_8); no longer J501.7 (Pin_7)
- net KNOB.RX: now also J501.9 (Pin_9); no longer J501.10 (Pin_10)
- net KNOB.SWCLK: now also J501.11 (Pin_11); no longer J501.12 (Pin_12)
- net KNOB.SWDIO: now also J501.12 (Pin_12); no longer J501.11 (Pin_11)
- net VBUS: now also J501.1 (Pin_1); no longer J501.2 (Pin_2)
- net ~{RST}: now also J501.4 (Pin_4); no longer J501.3 (Pin_3)
Other:
- moved on the sheet: J501
Changed lines of the file:
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@@
 	(symbol
 		(lib_id "Connector_Generic:Conn_02x08_Odd_Even")
-		(at 200.66 104.14 0)
-		(mirror x)
+		(at 203.2 104.14 180)
 		(unit 1)
 		(exclude_from_sim no)
@@
 		)
 		(property "Footprint" "Connector_PinHeader_1.27mm:PinHeader_2x08_P1.27mm_Horizontal"
-			(at 200.66 104.14 0)
+			(at 203.2 104.14 0)
 			(effects
 				(font
@@
 		)
 		(property "Datasheet" "~"
-			(at 200.66 104.14 0)
+			(at 203.2 104.14 0)
 			(effects
 				(font
@@
 		)
 		(property "Description" "Generic connector, double row, 02x08, odd/even pin numbering scheme (row 1 odd numbers, row 2 even numbers), script generated (kicad-library-utils/schlib/autogen/connector/)"
-			(at 200.66 104.14 0)
+			(at 203.2 104.14 0)
 			(effects
 				(font
