File: PCBs/keyboard-v3/fpc/fpc.kicad_pcb (KiCad board)
At the start: 2 copper layers, 72.4 x 19.3 mm, 0 parts

Commit message: Keyboard v3 hardware done
Routing:
- net RST: track 4.93 -> 2.47 mm, vias 2 -> 1
- net +5V: track 53.2 -> 55.6 mm, vias 4 -> 5
