File: PCBs/keyboard-v3/left-knob-board/left-knob-board.kicad_pcb (KiCad board)
At the start: 2 copper layers, 59 x 59 mm, 39 parts, among them J1 F31L-1A7H1-11008, M1 2206-100T, Q1 DMP21D0UFB-7B, Q2 DMN21D2UFB-7B, Q3 DMP21D0UFB-7B, SW1 SW_DIP_x01, SW2 SW_DIP_x01, SW3 SW_DIP_x01, U1 AS5600, U2 TMC6300-LA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

Commit message: Keyboard v3 hardware done
Other:
- board text added: "Keyboard v3 Left Knob Board Ben Smith 2026"
Changed lines of the file:
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@@
 			(sketchdnponfab yes)
 			(crossoutdnponfab yes)
-			(subtractmaskfromsilk no)
+			(subtractmaskfromsilk yes)
 			(outputformat 1)
 			(mirror no)
@@
 		)
 		(property "Height" "2.55"
-			(at 0 0 -90)
+			(at 0 0 270)
 			(unlocked yes)
 			(layer "B.Fab")
@@
 		(embedded_fonts no)
 	)
+	(gr_circle
+		(center 174 98)
+		(end 174 100)
+		(stroke
+			(width 0.1)
+			(type default)
+		)
+		(fill no)
+		(layer "F.SilkS")
+	)
 	(gr_line
 		(start 142.2 106.1)
@@
 		(layer "F.SilkS")
 	)
+	(gr_circle
+		(center 137.9 67)
+		(end 138.1 67)
+		(stroke
+			(width 0)
+			(type solid)
+		)
+		(fill yes)
+		(layer "F.SilkS")
+	)
 	(gr_line
 		(start 142.2 105.8)
@@
 		(layer "F.SilkS")
 	)
+	(gr_circle
+		(center 138 109.5)
+		(end 138 111.5)
+		(stroke
+			(width 0.1)
+			(type default)
+		)
+		(fill no)
+		(layer "F.SilkS")
+	)
+	(gr_circle
+		(center 140 75)
+		(end 140 77)
+		(stroke
+			(width 0.1)
+			(type default)
+		)
+		(fill no)
+		(layer "F.SilkS")
+	)
 	(gr_line
 		(start 143.8 106.1)
@@
 	)
 	(gr_circle
+		(center 145.6 67)
+		(end 145.8 67)
+		(stroke
+			(width 0)
+			(type solid)
+		)
+		(fill yes)
+		(layer "B.SilkS")
+	)
+	(gr_circle
+		(center 157 74)
+		(end 157 72)
+		(stroke
+			(width 0.1)
+			(type default)
+		)
+		(fill no)
+		(layer "B.SilkS")
+	)
+	(gr_circle
+		(center 151 80)
+		(end 151 78)
+		(stroke
+			(width 0.1)
+			(type default)
+		)
+		(fill no)
+		(layer "B.SilkS")
+	)
+	(gr_circle
+		(center 163 80)
+		(end 163 78)
+		(stroke
+			(width 0.1)
+			(type default)
+		)
+		(fill no)
+		(layer "B.SilkS")
+	)
+	(gr_circle
+		(center 157 86)
+		(end 157 84)
+		(stroke
+			(width 0.1)
+			(type default)
+		)
+		(fill no)
+		(layer "B.SilkS")
+	)
+	(gr_circle
 		(center 157 80)
 		(end 138 80)
@@
 		)
 	)
+	(gr_text "Keyboard v3\nLeft Knob Board\nBen Smith 2026"
+		(at 165.4 69 0)
+		(layer "B.SilkS")
+		(effects
+			(font
+				(size 1 1)
+				(thickness 0.1)
+			)
+			(justify mirror)
+		)
+	)
